File: hardware/PCB_Aquarium2/HC05.kicad_sch (KiCad schematic)
At the start: 1 part, among them J39 Conn_01x04

Commit message: PCBs v3
Parts:
- added C38: 1u, Capacitor_SMD:C_0603_1608Metric, symbol Device:C
Connections:
- net +5V: now also C38.1; no longer J39.1 (Pin_1)
- new net: C38.2, J39.1 (Pin_1)
Changed lines of the file:
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@@
 	(wire
 		(pts
-			(xy 135.89 83.82) (xy 139.7 83.82)
+			(xy 138.43 83.82) (xy 139.7 83.82)
+		)
+		(stroke
+			(width 0)
+			(type default)
+		)
+	)
+	(wire
+		(pts
+			(xy 129.54 83.82) (xy 130.81 83.82)
 		)
 		(stroke
@@
 	)
 	(symbol
+		(lib_id "Device:C")
+		(at 134.62 83.82 90)
+		(unit 1)
+		(exclude_from_sim no)
+		(in_bom yes)
+		(on_board yes)
+		(dnp no)
+		(fields_autoplaced yes)
+		(property "Reference" "C38"
+			(at 134.62 76.2 90)
+			(effects
+				(font
+					(size 1.27 1.27)
+				)
+			)
+		)
+		(property "Value" "1u"
+			(at 134.62 78.74 90)
+			(effects
+				(font
+					(size 1.27 1.27)
+				)
+			)
+		)
+		(property "Footprint" "Capacitor_SMD:C_0603_1608Metric"
+			(at 138.43 82.8548 0)
+			(effects
+				(font
+					(size 1.27 1.27)
+				)
+				(hide yes)
+			)
+		)
+		(property "Datasheet" "~"
+			(at 134.62 83.82 0)
+			(effects
+				(font
+					(size 1.27 1.27)
+				)
+				(hide yes)
+			)
+		)
+		(property "Description" "Unpolarized capacitor"
+			(at 134.62 83.82 0)
+			(effects
+				(font
+					(size 1.27 1.27)
+				)
+				(hide yes)
+			)
+		)
+		(pin "2"
+		)
+		(pin "1"
+		)
+		(instances
+			(project ""
+				(path "/4f9429d5-fbb3-48e9-90dd-7ff0c2950e6f/25085fa0-d3fc-4eed-8ed3-1cfc9369e5eb"
+					(reference "C38")
+					(unit 1)
+				)
+			)
+		)
+	)
+	(symbol
 		(lib_name "+5V_1")
 		(lib_id "power:+5V")
-		(at 135.89 83.82 90)
+		(at 129.54 83.82 0)
 		(unit 1)
 		(exclude_from_sim no)
@@
 		(fields_autoplaced yes)
 		(property "Reference" "#PWR092"
-			(at 139.7 83.82 0)
+			(at 129.54 87.63 0)
 			(effects
 				(font
@@
 		)
 		(property "Value" "+5V"
-			(at 132.08 83.8199 90)
+			(at 129.54 78.74 0)
 			(effects
 				(font
 					(size 1.27 1.27)
 				)
-				(justify left)
 			)
 		)
 		(property "Footprint" ""
-			(at 135.89 83.82 0)
+			(at 129.54 83.82 0)
 			(effects
 				(font
@@
 		)
 		(property "Datasheet" ""
-			(at 135.89 83.82 0)
+			(at 129.54 83.82 0)
 			(effects
 				(font
@@
 		)
 		(property "Description" "Power symbol creates a global label with name \"+5V\""
-			(at 135.89 83.82 0)
+			(at 129.54 83.82 0)
 			(effects
 				(font

Commit message: PCBs v4
Parts:
- renumbered C38 to C44, J39 to J38
Connections:
- net +5V: now also C44.2, J38.1 (Pin_1); no longer C44.1
- net GND: now also C44.1
Other:
- moved on the sheet: C44
Changed lines of the file:
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@@
 	(generator_version "9.0")
 	(paper "A4")
-	(wire
-		(pts
-			(xy 135.89 86.36) (xy 139.7 86.36)
+	(junction
+		(at 134.62 86.36)
+		(diameter 0)
+		(color 0 0 0 0)
+	)
+	(junction
+		(at 134.62 78.74)
+		(diameter 0)
+		(color 0 0 0 0)
+	)
+	(wire
+		(pts
+			(xy 130.81 86.36) (xy 134.62 86.36)
 		)
 		(stroke
@@
 	(wire
 		(pts
+			(xy 138.43 78.74) (xy 134.62 78.74)
+		)
+		(stroke
+			(width 0)
+			(type default)
+		)
+	)
+	(wire
+		(pts
 			(xy 135.89 91.44) (xy 139.7 91.44)
 		)
@@
 	(wire
 		(pts
+			(xy 138.43 83.82) (xy 138.43 78.74)
+		)
+		(stroke
+			(width 0)
+			(type default)
+		)
+	)
+	(wire
+		(pts
+			(xy 134.62 86.36) (xy 139.7 86.36)
+		)
+		(stroke
+			(width 0)
+			(type default)
+		)
+	)
+	(wire
+		(pts
 			(xy 138.43 83.82) (xy 139.7 83.82)
 		)
@@
 	(wire
 		(pts
-			(xy 129.54 83.82) (xy 130.81 83.82)
+			(xy 129.54 78.74) (xy 134.62 78.74)
 		)
 		(stroke
@@
 	(symbol
 		(lib_id "Device:C")
-		(at 134.62 83.82 90)
+		(at 134.62 82.55 180)
 		(unit 1)
 		(exclude_from_sim no)
@@
 		(dnp no)
 		(fields_autoplaced yes)
-		(property "Reference" "C38"
-			(at 134.62 76.2 90)
-			(effects
-				(font
-					(size 1.27 1.27)
-				)
+		(property "Reference" "C44"
+			(at 138.43 81.2799 0)
+			(effects
+				(font
+					(size 1.27 1.27)
+				)
+				(justify right)
 			)
 		)
 		(property "Value" "1u"
-			(at 134.62 78.74 90)
-			(effects
-				(font
-					(size 1.27 1.27)
-				)
+			(at 138.43 83.8199 0)
+			(effects
+				(font
+					(size 1.27 1.27)
+				)
+				(justify right)
 			)
 		)
 		(property "Footprint" "Capacitor_SMD:C_0603_1608Metric"
-			(at 138.43 82.8548 0)
+			(at 133.6548 78.74 0)
 			(effects
 				(font
@@
 		)
 		(property "Datasheet" "~"
-			(at 134.62 83.82 0)
+			(at 134.62 82.55 0)
 			(effects
 				(font
@@
 		)
 		(property "Description" "Unpolarized capacitor"
-			(at 134.62 83.82 0)
+			(at 134.62 82.55 0)
 			(effects
 				(font
@@
 		)
 		(instances
-			(project ""
+			(project "PCB_Aquarium2"
 				(path "/4f9429d5-fbb3-48e9-90dd-7ff0c2950e6f/25085fa0-d3fc-4eed-8ed3-1cfc9369e5eb"
-					(reference "C38")
+					(reference "C44")
 					(unit 1)
 				)
@@
 		(lib_name "+5V_1")
 		(lib_id "power:+5V")
-		(at 129.54 83.82 0)
+		(at 129.54 78.74 0)
 		(unit 1)
 		(exclude_from_sim no)
@@
 		(dnp no)
 		(fields_autoplaced yes)
-		(property "Reference" "#PWR092"
-			(at 129.54 87.63 0)
+		(property "Reference" "#PWR090"
+			(at 129.54 82.55 0)
 			(effects
 				(font
@@
 		)
 		(property "Value" "+5V"
+			(at 129.54 73.66 0)
+			(effects
+				(font
+					(size 1.27 1.27)
+				)
+			)
+		)
+		(property "Footprint" ""
 			(at 129.54 78.74 0)
 			(effects
@@
 					(size 1.27 1.27)
 				)
-			)
-		)
-		(property "Footprint" ""
-			(at 129.54 83.82 0)
-			(effects
-				(font
-					(size 1.27 1.27)
-				)
 				(hide yes)
 			)
 		)
 		(property "Datasheet" ""
-			(at 129.54 83.82 0)
+			(at 129.54 78.74 0)
 			(effects
 				(font
@@
 		)
 		(property "Description" "Power symbol creates a global label with name \"+5V\""
-			(at 129.54 83.82 0)
+			(at 129.54 78.74 0)
 			(effects
 				(font
@@
 			(project "PCB_Aquarium2"
 				(path "/4f9429d5-fbb3-48e9-90dd-7ff0c2950e6f/25085fa0-d3fc-4eed-8ed3-1cfc9369e5eb"
-					(reference "#PWR092")
+					(reference "#PWR090")
 					(unit 1)
 				)
@@
 		(lib_name "GND_2")
 		(lib_id "power:GND")
-		(at 135.89 86.36 270)
+		(at 130.81 86.36 270)
 		(unit 1)
 		(exclude_from_sim no)
@@
 		(dnp no)
 		(fields_autoplaced yes)
-		(property "Reference" "#PWR093"
-			(at 129.54 86.36 0)
+		(property "Reference" "#PWR091"
+			(at 124.46 86.36 0)
 			(effects
 				(font
@@
 		)
 		(property "Value" "GND"
-			(at 132.08 86.3599 90)
+			(at 127 86.3599 90)
 			(effects
 				(font
@@
 		)
 		(property "Footprint" ""
-			(at 135.89 86.36 0)
+			(at 130.81 86.36 0)
 			(effects
 				(font
@@
 		)
 		(property "Datasheet" ""
-			(at 135.89 86.36 0)
+			(at 130.81 86.36 0)
 			(effects
 				(font
@@
 		)
 		(property "Description" "Power symbol creates a global label with name \"GND\" , ground"
-			(at 135.89 86.36 0)
+			(at 130.81 86.36 0)
 			(effects
 				(font
@@
 			(project "PCB_Aquarium2"
 				(path "/4f9429d5-fbb3-48e9-90dd-7ff0c2950e6f/25085fa0-d3fc-4eed-8ed3-1cfc9369e5eb"
-					(reference "#PWR093")
+					(reference "#PWR091")
 					(unit 1)
 				)
@@
 		(dnp no)
 		(fields_autoplaced yes)
-		(property "Reference" "J39"
+		(property "Reference" "J38"
 			(at 147.32 86.3599 0)
 			(effects
@@
 			(project "PCB_Aquarium2"
 				(path "/4f9429d5-fbb3-48e9-90dd-7ff0c2950e6f/25085fa0-d3fc-4eed-8ed3-1cfc9369e5eb"
-					(reference "J39")
+					(reference "J38")
 					(unit 1)
 				)
