File: hardware/PCB_Aquarium2/LED_internes.kicad_sch (KiCad schematic)
At the start: 1 part, among them J37 Conn_01x03

Commit message: PCBs v3
Parts:
- added C35: 1u, Capacitor_SMD:C_0603_1608Metric, symbol Device:C
Connections:
- net +5V: now also C35.1; no longer J37.1 (Pin_1)
- new net: C35.2, J37.1 (Pin_1)
Changed lines of the file:
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@@
+	(wire
+		(pts
+			(xy 127 88.9) (xy 128.27 88.9)
+		)
+		(stroke
+			(width 0)
+			(type default)
+		)
+	)
 	(wire
 		(pts
@@
 	(wire
 		(pts
-			(xy 134.62 88.9) (xy 137.16 88.9)
+			(xy 135.89 88.9) (xy 137.16 88.9)
 		)
 		(stroke
@@
 	(symbol
 		(lib_id "power:+5V")
-		(at 134.62 88.9 0)
+		(at 127 88.9 0)
 		(unit 1)
 		(exclude_from_sim no)
@@
 		(fields_autoplaced yes)
 		(property "Reference" "#PWR088"
-			(at 134.62 92.71 0)
+			(at 127 92.71 0)
 			(effects
 				(font
@@
 		)
 		(property "Value" "+5V"
-			(at 134.62 83.82 0)
+			(at 127 83.82 0)
 			(effects
 				(font
@@
 		)
 		(property "Footprint" ""
-			(at 134.62 88.9 0)
+			(at 127 88.9 0)
 			(effects
 				(font
@@
 		)
 		(property "Datasheet" ""
-			(at 134.62 88.9 0)
+			(at 127 88.9 0)
 			(effects
 				(font
@@
 		)
 		(property "Description" "Power symbol creates a global label with name \"+5V\""
-			(at 134.62 88.9 0)
+			(at 127 88.9 0)
 			(effects
 				(font
@@
 					(unit 1)
 				)
+			)
+		)
+	)
+	(symbol
+		(lib_id "Device:C")
+		(at 132.08 88.9 90)
+		(unit 1)
+		(exclude_from_sim no)
+		(in_bom yes)
+		(on_board yes)
+		(dnp no)
+		(fields_autoplaced yes)
+		(property "Reference" "C35"
+			(at 132.08 81.28 90)
+			(effects
+				(font
+					(size 1.27 1.27)
+				)
+			)
+		)
+		(property "Value" "1u"
+			(at 132.08 83.82 90)
+			(effects
+				(font
+					(size 1.27 1.27)
+				)
+			)
+		)
+		(property "Footprint" "Capacitor_SMD:C_0603_1608Metric"
+			(at 135.89 87.9348 0)
+			(effects
+				(font
+					(size 1.27 1.27)
+				)
+				(hide yes)
+			)
+		)
+		(property "Datasheet" "~"
+			(at 132.08 88.9 0)
+			(effects
+				(font
+					(size 1.27 1.27)
+				)
+				(hide yes)
+			)
+		)
+		(property "Description" "Unpolarized capacitor"
+			(at 132.08 88.9 0)
+			(effects
+				(font
+					(size 1.27 1.27)
+				)
+				(hide yes)
+			)
+		)
+		(pin "1"
+		)
+		(pin "2"
+		)
+		(instances
+			(project ""
+				(path "/4f9429d5-fbb3-48e9-90dd-7ff0c2950e6f/9b3ea6c7-576b-4238-ae95-35be57471754"
+					(reference "C35")
+					(unit 1)
+				)

Commit message: PCBs v4
Parts:
- renumbered C35 to C42, J37 to J36
Connections:
- net +5V: now also C42.2, J36.1 (Pin_1); no longer C42.1
- net GND: now also C42.1
Other:
- moved on the sheet: C42
Changed lines of the file:
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@@
 	(generator_version "9.0")
 	(paper "A4")
-	(wire
-		(pts
-			(xy 127 88.9) (xy 128.27 88.9)
+	(junction
+		(at 127 87.63)
+		(diameter 0)
+		(color 0 0 0 0)
+	)
+	(junction
+		(at 127 95.25)
+		(diameter 0)
+		(color 0 0 0 0)
+	)
+	(wire
+		(pts
+			(xy 137.16 95.25) (xy 137.16 93.98)
+		)
+		(stroke
+			(width 0)
+			(type default)
+		)
+	)
+	(wire
+		(pts
+			(xy 123.19 87.63) (xy 127 87.63)
 		)
 		(stroke
@@
 	(wire
 		(pts
-			(xy 134.62 93.98) (xy 137.16 93.98)
-		)
-		(stroke
-			(width 0)
-			(type default)
-		)
-	)
-	(wire
-		(pts
-			(xy 135.89 88.9) (xy 137.16 88.9)
+			(xy 137.16 87.63) (xy 137.16 88.9)
+		)
+		(stroke
+			(width 0)
+			(type default)
+		)
+	)
+	(wire
+		(pts
+			(xy 124.46 95.25) (xy 127 95.25)
+		)
+		(stroke
+			(width 0)
+			(type default)
+		)
+	)
+	(wire
+		(pts
+			(xy 127 95.25) (xy 137.16 95.25)
+		)
+		(stroke
+			(width 0)
+			(type default)
+		)
+	)
+	(wire
+		(pts
+			(xy 127 87.63) (xy 137.16 87.63)
 		)
 		(stroke
@@
 	(symbol
 		(lib_id "power:+5V")
-		(at 127 88.9 0)
+		(at 123.19 87.63 0)
 		(unit 1)
 		(exclude_from_sim no)
@@
 		(dnp no)
 		(fields_autoplaced yes)
-		(property "Reference" "#PWR088"
-			(at 127 92.71 0)
+		(property "Reference" "#PWR086"
+			(at 123.19 91.44 0)
 			(effects
 				(font
@@
 		)
 		(property "Value" "+5V"
-			(at 127 83.82 0)
+			(at 123.19 82.55 0)
 			(effects
 				(font
@@
 		)
 		(property "Footprint" ""
-			(at 127 88.9 0)
+			(at 123.19 87.63 0)
 			(effects
 				(font
@@
 		)
 		(property "Datasheet" ""
-			(at 127 88.9 0)
+			(at 123.19 87.63 0)
 			(effects
 				(font
@@
 		)
 		(property "Description" "Power symbol creates a global label with name \"+5V\""
-			(at 127 88.9 0)
+			(at 123.19 87.63 0)
 			(effects
 				(font
@@
 			(project ""
 				(path "/4f9429d5-fbb3-48e9-90dd-7ff0c2950e6f/9b3ea6c7-576b-4238-ae95-35be57471754"
-					(reference "#PWR088")
+					(reference "#PWR086")
 					(unit 1)
 				)
@@
 	(symbol
 		(lib_id "power:GND")
-		(at 134.62 93.98 0)
+		(at 124.46 95.25 0)
 		(unit 1)
 		(exclude_from_sim no)
@@
 		(dnp no)
 		(fields_autoplaced yes)
-		(property "Reference" "#PWR089"
-			(at 134.62 100.33 0)
+		(property "Reference" "#PWR087"
+			(at 124.46 101.6 0)
 			(effects
 				(font
@@
 		)
 		(property "Value" "GND"
-			(at 134.62 99.06 0)
+			(at 124.46 100.33 0)
 			(effects
 				(font
@@
 		)
 		(property "Footprint" ""
-			(at 134.62 93.98 0)
+			(at 124.46 95.25 0)
 			(effects
 				(font
@@
 		)
 		(property "Datasheet" ""
-			(at 134.62 93.98 0)
+			(at 124.46 95.25 0)
 			(effects
 				(font
@@
 		)
 		(property "Description" "Power symbol creates a global label with name \"GND\" , ground"
-			(at 134.62 93.98 0)
+			(at 124.46 95.25 0)
 			(effects
 				(font
@@
 			(project ""
 				(path "/4f9429d5-fbb3-48e9-90dd-7ff0c2950e6f/9b3ea6c7-576b-4238-ae95-35be57471754"
-					(reference "#PWR089")
+					(reference "#PWR087")
 					(unit 1)
 				)
@@
 	(symbol
 		(lib_id "Device:C")
-		(at 132.08 88.9 90)
+		(at 127 91.44 180)
 		(unit 1)
 		(exclude_from_sim no)
@@
 		(dnp no)
 		(fields_autoplaced yes)
-		(property "Reference" "C35"
-			(at 132.08 81.28 90)
-			(effects
-				(font
-					(size 1.27 1.27)
-				)
+		(property "Reference" "C42"
+			(at 130.81 90.1699 0)
+			(effects
+				(font
+					(size 1.27 1.27)
+				)
+				(justify right)
 			)
 		)
 		(property "Value" "1u"
-			(at 132.08 83.82 90)
-			(effects
-				(font
-					(size 1.27 1.27)
-				)
+			(at 130.81 92.7099 0)
+			(effects
+				(font
+					(size 1.27 1.27)
+				)
+				(justify right)
 			)
 		)
 		(property "Footprint" "Capacitor_SMD:C_0603_1608Metric"
-			(at 135.89 87.9348 0)
+			(at 126.0348 87.63 0)
 			(effects
 				(font
@@
 		)
 		(property "Datasheet" "~"
-			(at 132.08 88.9 0)
+			(at 127 91.44 0)
 			(effects
 				(font
@@
 		)
 		(property "Description" "Unpolarized capacitor"
-			(at 132.08 88.9 0)
+			(at 127 91.44 0)
 			(effects
 				(font
@@
 		)
 		(instances
-			(project ""
+			(project "PCB_Aquarium2"
 				(path "/4f9429d5-fbb3-48e9-90dd-7ff0c2950e6f/9b3ea6c7-576b-4238-ae95-35be57471754"
-					(reference "C35")
+					(reference "C42")
 					(unit 1)
 				)
@@
 		(dnp no)
 		(fields_autoplaced yes)
-		(property "Reference" "J37"
+		(property "Reference" "J36"
 			(at 144.78 90.1699 0)
 			(effects
@@
 			(project "PCB_Aquarium2"
 				(path "/4f9429d5-fbb3-48e9-90dd-7ff0c2950e6f/9b3ea6c7-576b-4238-ae95-35be57471754"
-					(reference "J37")
+					(reference "J36")
 					(unit 1)
 				)
