File: hardware/PCB_Aquarium2/PH_meter.kicad_sch (KiCad schematic)
At the start: 1 part, among them J1 Conn_01x03

Commit message: PCBs v3
Parts:
- added C28: 1u, Capacitor_SMD:C_0603_1608Metric, symbol Device:C
Connections:
- net +5V: now also C28.1; no longer J1.2 (Pin_2)
- new net: C28.2, J1.2 (Pin_2)
Changed lines of the file:
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@@
 	(wire
 		(pts
-			(xy 128.27 101.6) (xy 137.16 101.6)
+			(xy 130.81 101.6) (xy 137.16 101.6)
+		)
+		(stroke
+			(width 0)
+			(type default)
+		)
+	)
+	(wire
+		(pts
+			(xy 120.65 101.6) (xy 123.19 101.6)
 		)
 		(stroke
@@
 	(symbol
 		(lib_id "power:+5V")
-		(at 128.27 101.6 0)
+		(at 120.65 101.6 0)
 		(unit 1)
 		(exclude_from_sim no)
@@
 		(fields_autoplaced yes)
 		(property "Reference" "#PWR08"
-			(at 128.27 105.41 0)
+			(at 120.65 105.41 0)
 			(effects
 				(font
@@
 		)
 		(property "Value" "+5V"
-			(at 128.27 96.52 0)
+			(at 120.65 96.52 0)
 			(effects
 				(font
@@
 		)
 		(property "Footprint" ""
-			(at 128.27 101.6 0)
+			(at 120.65 101.6 0)
 			(effects
 				(font
@@
 		)
 		(property "Datasheet" ""
-			(at 128.27 101.6 0)
+			(at 120.65 101.6 0)
 			(effects
 				(font
@@
 		)
 		(property "Description" "Power symbol creates a global label with name \"+5V\""
-			(at 128.27 101.6 0)
+			(at 120.65 101.6 0)
 			(effects
 				(font
@@
 					(unit 1)
 				)
+			)
+		)
+	)
+	(symbol
+		(lib_id "Device:C")
+		(at 127 101.6 90)
+		(unit 1)
+		(exclude_from_sim no)
+		(in_bom yes)
+		(on_board yes)
+		(dnp no)
+		(fields_autoplaced yes)
+		(property "Reference" "C28"
+			(at 127 93.98 90)
+			(effects
+				(font
+					(size 1.27 1.27)
+				)
+			)
+		)
+		(property "Value" "1u"
+			(at 127 96.52 90)
+			(effects
+				(font
+					(size 1.27 1.27)
+				)
+			)
+		)
+		(property "Footprint" "Capacitor_SMD:C_0603_1608Metric"
+			(at 130.81 100.6348 0)
+			(effects
+				(font
+					(size 1.27 1.27)
+				)
+				(hide yes)
+			)
+		)
+		(property "Datasheet" "~"
+			(at 127 101.6 0)
+			(effects
+				(font
+					(size 1.27 1.27)
+				)
+				(hide yes)
+			)
+		)
+		(property "Description" "Unpolarized capacitor"
+			(at 127 101.6 0)
+			(effects
+				(font
+					(size 1.27 1.27)
+				)
+				(hide yes)
+			)
+		)
+		(pin "1"
+		)
+		(pin "2"
+		)
+		(instances
+			(project ""
+				(path "/4f9429d5-fbb3-48e9-90dd-7ff0c2950e6f/93cb062e-b48a-4ff4-9534-f1dcb451c7c1"
+					(reference "C28")
+					(unit 1)
+				)

Commit message: PCBs v4
Parts:
- renumbered C28 to C11
Connections:
- net +5V: now also J1.2 (Pin_2)
- net GND: now also C11.2
Other:
- moved on the sheet: C11
Changed lines of the file:
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@@
 	(generator_version "9.0")
 	(paper "A4")
+	(junction
+		(at 128.27 93.98)
+		(diameter 0)
+		(color 0 0 0 0)
+	)
+	(junction
+		(at 128.27 101.6)
+		(diameter 0)
+		(color 0 0 0 0)
+	)
+	(wire
+		(pts
+			(xy 132.08 93.98) (xy 132.08 99.06)
+		)
+		(stroke
+			(width 0)
+			(type default)
+		)
+	)
+	(wire
+		(pts
+			(xy 128.27 93.98) (xy 132.08 93.98)
+		)
+		(stroke
+			(width 0)
+			(type default)
+		)
+	)
+	(wire
+		(pts
+			(xy 123.19 93.98) (xy 128.27 93.98)
+		)
+		(stroke
+			(width 0)
+			(type default)
+		)
+	)
+	(wire
+		(pts
+			(xy 120.65 101.6) (xy 128.27 101.6)
+		)
+		(stroke
+			(width 0)
+			(type default)
+		)
+	)
 	(wire
 		(pts
@@
 	(wire
 		(pts
-			(xy 130.81 101.6) (xy 137.16 101.6)
-		)
-		(stroke
-			(width 0)
-			(type default)
-		)
-	)
-	(wire
-		(pts
-			(xy 120.65 101.6) (xy 123.19 101.6)
+			(xy 128.27 101.6) (xy 137.16 101.6)
 		)
 		(stroke
@@
 	(symbol
 		(lib_id "Device:C")
-		(at 127 101.6 90)
+		(at 128.27 97.79 180)
 		(unit 1)
 		(exclude_from_sim no)
@@
 		(dnp no)
 		(fields_autoplaced yes)
-		(property "Reference" "C28"
-			(at 127 93.98 90)
-			(effects
-				(font
-					(size 1.27 1.27)
-				)
+		(property "Reference" "C11"
+			(at 132.08 96.5199 0)
+			(effects
+				(font
+					(size 1.27 1.27)
+				)
+				(justify right)
 			)
 		)
 		(property "Value" "1u"
-			(at 127 96.52 90)
-			(effects
-				(font
-					(size 1.27 1.27)
-				)
+			(at 132.08 99.0599 0)
+			(effects
+				(font
+					(size 1.27 1.27)
+				)
+				(justify right)
 			)
 		)
 		(property "Footprint" "Capacitor_SMD:C_0603_1608Metric"
-			(at 130.81 100.6348 0)
+			(at 127.3048 93.98 0)
 			(effects
 				(font
@@
 		)
 		(property "Datasheet" "~"
-			(at 127 101.6 0)
+			(at 128.27 97.79 0)
 			(effects
 				(font
@@
 		)
 		(property "Description" "Unpolarized capacitor"
-			(at 127 101.6 0)
+			(at 128.27 97.79 0)
 			(effects
 				(font
@@
 		)
 		(instances
-			(project ""
+			(project "PCB_Aquarium2"
 				(path "/4f9429d5-fbb3-48e9-90dd-7ff0c2950e6f/93cb062e-b48a-4ff4-9534-f1dcb451c7c1"
-					(reference "C28")
+					(reference "C11")
 					(unit 1)
 				)
@@
 	(symbol
 		(lib_id "power:GND")
-		(at 132.08 99.06 180)
+		(at 123.19 93.98 180)
 		(unit 1)
 		(exclude_from_sim no)
@@
 		(fields_autoplaced yes)
 		(property "Reference" "#PWR09"
-			(at 132.08 92.71 0)
+			(at 123.19 87.63 0)
 			(effects
 				(font
@@
 		)
 		(property "Value" "GND"
-			(at 132.08 93.98 0)
+			(at 123.19 88.9 0)
 			(effects
 				(font
@@
 		)
 		(property "Footprint" ""
-			(at 132.08 99.06 0)
+			(at 123.19 93.98 0)
 			(effects
 				(font
@@
 		)
 		(property "Datasheet" ""
-			(at 132.08 99.06 0)
+			(at 123.19 93.98 0)
 			(effects
 				(font
@@
 		)
 		(property "Description" "Power symbol creates a global label with name \"GND\" , ground"
-			(at 132.08 99.06 0)
-			(effects
-				(font
+			(at 123.19 93.98 0)
+			(effects
+				(font
