File: hardware/PCB_Aquarium2/RasberryPi4.kicad_sch (KiCad schematic)
At the start: 1 part, among them J35 Conn_01x04

Commit message: PCBs v3
Parts:
- added C37: 1u, Capacitor_SMD:C_0603_1608Metric, symbol Device:C
Connections:
- net +5V: now also C37.1; no longer J35.1 (Pin_1)
- new net: C37.2, J35.1 (Pin_1)
Changed lines of the file:
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@@
 	(wire
 		(pts
-			(xy 140.97 83.82) (xy 142.24 83.82)
-		)
-		(stroke
-			(width 0)
-			(type default)
-		)
-	)
-	(wire
-		(pts
-			(xy 134.62 86.36) (xy 142.24 86.36)
+			(xy 128.27 86.36) (xy 142.24 86.36)
 		)
 		(stroke
@@
 	)
 	(symbol
+		(lib_id "Device:C")
+		(at 138.43 83.82 90)
+		(unit 1)
+		(exclude_from_sim no)
+		(in_bom yes)
+		(on_board yes)
+		(dnp no)
+		(fields_autoplaced yes)
+		(property "Reference" "C37"
+			(at 138.43 76.2 90)
+			(effects
+				(font
+					(size 1.27 1.27)
+				)
+			)
+		)
+		(property "Value" "1u"
+			(at 138.43 78.74 90)
+			(effects
+				(font
+					(size 1.27 1.27)
+				)
+			)
+		)
+		(property "Footprint" "Capacitor_SMD:C_0603_1608Metric"
+			(at 142.24 82.8548 0)
+			(effects
+				(font
+					(size 1.27 1.27)
+				)
+				(hide yes)
+			)
+		)
+		(property "Datasheet" "~"
+			(at 138.43 83.82 0)
+			(effects
+				(font
+					(size 1.27 1.27)
+				)
+				(hide yes)
+			)
+		)
+		(property "Description" "Unpolarized capacitor"
+			(at 138.43 83.82 0)
+			(effects
+				(font
+					(size 1.27 1.27)
+				)
+				(hide yes)
+			)
+		)
+		(pin "2"
+		)
+		(pin "1"
+		)
+		(instances
+			(project ""
+				(path "/4f9429d5-fbb3-48e9-90dd-7ff0c2950e6f/6b08732c-65b5-4020-967e-cc3e23d6bed3"
+					(reference "C37")
+					(unit 1)
+				)
+			)
+		)
+	)
+	(symbol
 		(lib_id "power:+5V")
-		(at 140.97 83.82 0)
+		(at 134.62 83.82 0)
 		(unit 1)
 		(exclude_from_sim no)
@@
 		(fields_autoplaced yes)
 		(property "Reference" "#PWR085"
-			(at 140.97 87.63 0)
+			(at 134.62 87.63 0)
 			(effects
 				(font
@@
 		)
 		(property "Value" "+5V"
-			(at 140.97 78.74 0)
+			(at 134.62 78.74 0)
 			(effects
 				(font
@@
 		)
 		(property "Footprint" ""
-			(at 140.97 83.82 0)
+			(at 134.62 83.82 0)
 			(effects
 				(font
@@
 		)
 		(property "Datasheet" ""
-			(at 140.97 83.82 0)
+			(at 134.62 83.82 0)
 			(effects
 				(font
@@
 		)
 		(property "Description" "Power symbol creates a global label with name \"+5V\""
-			(at 140.97 83.82 0)
+			(at 134.62 83.82 0)
 			(effects
 				(font
@@
 	(symbol
 		(lib_id "power:GND")
-		(at 134.62 86.36 180)
+		(at 128.27 86.36 180)
 		(unit 1)
 		(exclude_from_sim no)
@@
 		(fields_autoplaced yes)
 		(property "Reference" "#PWR084"
-			(at 134.62 80.01 0)
+			(at 128.27 80.01 0)
 			(effects
 				(font
@@
 		)
 		(property "Value" "GND"
-			(at 134.62 81.28 0)
+			(at 128.27 81.28 0)
 			(effects
 				(font
@@
 		)
 		(property "Footprint" ""
-			(at 134.62 86.36 0)
+			(at 128.27 86.36 0)
 			(effects
 				(font
@@
 		)
 		(property "Datasheet" ""
-			(at 134.62 86.36 0)
+			(at 128.27 86.36 0)
 			(effects
 				(font
@@
 		)
 		(property "Description" "Power symbol creates a global label with name \"GND\" , ground"
-			(at 134.62 86.36 0)
-			(effects
-				(font
+			(at 128.27 86.36 0)
+			(effects
+				(font

Commit message: PCBs v4
Parts:
- renumbered C37 to C41, J35 to J34
Connections:
- net +5V: now also C41.2, J34.1 (Pin_1); no longer C41.1
- net GND: now also C41.1
Other:
- moved on the sheet: C41
Changed lines of the file:
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@@
 	(generator_version "9.0")
 	(paper "A4")
-	(wire
-		(pts
-			(xy 128.27 86.36) (xy 142.24 86.36)
+	(junction
+		(at 135.89 78.74)
+		(diameter 0)
+		(color 0 0 0 0)
+	)
+	(junction
+		(at 135.89 86.36)
+		(diameter 0)
+		(color 0 0 0 0)
+	)
+	(wire
+		(pts
+			(xy 135.89 86.36) (xy 142.24 86.36)
+		)
+		(stroke
+			(width 0)
+			(type default)
+		)
+	)
+	(wire
+		(pts
+			(xy 128.27 86.36) (xy 135.89 86.36)
+		)
+		(stroke
+			(width 0)
+			(type default)
+		)
+	)
+	(wire
+		(pts
+			(xy 142.24 78.74) (xy 135.89 78.74)
+		)
+		(stroke
+			(width 0)
+			(type default)
+		)
+	)
+	(wire
+		(pts
+			(xy 135.89 78.74) (xy 133.35 78.74)
+		)
+		(stroke
+			(width 0)
+			(type default)
+		)
+	)
+	(wire
+		(pts
+			(xy 142.24 83.82) (xy 142.24 78.74)
 		)
 		(stroke
@@
 	(symbol
 		(lib_id "Device:C")
-		(at 138.43 83.82 90)
+		(at 135.89 82.55 180)
 		(unit 1)
 		(exclude_from_sim no)
@@
 		(dnp no)
 		(fields_autoplaced yes)
-		(property "Reference" "C37"
-			(at 138.43 76.2 90)
-			(effects
-				(font
-					(size 1.27 1.27)
-				)
+		(property "Reference" "C41"
+			(at 139.7 81.2799 0)
+			(effects
+				(font
+					(size 1.27 1.27)
+				)
+				(justify right)
 			)
 		)
 		(property "Value" "1u"
-			(at 138.43 78.74 90)
-			(effects
-				(font
-					(size 1.27 1.27)
-				)
+			(at 139.7 83.8199 0)
+			(effects
+				(font
+					(size 1.27 1.27)
+				)
+				(justify right)
 			)
 		)
 		(property "Footprint" "Capacitor_SMD:C_0603_1608Metric"
-			(at 142.24 82.8548 0)
+			(at 134.9248 78.74 0)
 			(effects
 				(font
@@
 		)
 		(property "Datasheet" "~"
-			(at 138.43 83.82 0)
+			(at 135.89 82.55 0)
 			(effects
 				(font
@@
 		)
 		(property "Description" "Unpolarized capacitor"
-			(at 138.43 83.82 0)
+			(at 135.89 82.55 0)
 			(effects
 				(font
@@
 		)
 		(instances
-			(project ""
+			(project "PCB_Aquarium2"
 				(path "/4f9429d5-fbb3-48e9-90dd-7ff0c2950e6f/6b08732c-65b5-4020-967e-cc3e23d6bed3"
-					(reference "C37")
+					(reference "C41")
 					(unit 1)
 				)
@@
 	(symbol
 		(lib_id "power:+5V")
-		(at 134.62 83.82 0)
+		(at 133.35 78.74 0)
 		(unit 1)
 		(exclude_from_sim no)
@@
 		(dnp no)
 		(fields_autoplaced yes)
-		(property "Reference" "#PWR085"
-			(at 134.62 87.63 0)
+		(property "Reference" "#PWR083"
+			(at 133.35 82.55 0)
 			(effects
 				(font
@@
 		)
 		(property "Value" "+5V"
-			(at 134.62 78.74 0)
+			(at 133.35 73.66 0)
 			(effects
 				(font
@@
 		)
 		(property "Footprint" ""
-			(at 134.62 83.82 0)
+			(at 133.35 78.74 0)
 			(effects
 				(font
@@
 		)
 		(property "Datasheet" ""
-			(at 134.62 83.82 0)
+			(at 133.35 78.74 0)
 			(effects
 				(font
@@
 		)
 		(property "Description" "Power symbol creates a global label with name \"+5V\""
-			(at 134.62 83.82 0)
+			(at 133.35 78.74 0)
 			(effects
 				(font
@@
 			(project ""
 				(path "/4f9429d5-fbb3-48e9-90dd-7ff0c2950e6f/6b08732c-65b5-4020-967e-cc3e23d6bed3"
-					(reference "#PWR085")
+					(reference "#PWR083")
 					(unit 1)
 				)
@@
 		(dnp no)
 		(fields_autoplaced yes)
-		(property "Reference" "J35"
+		(property "Reference" "J34"
 			(at 149.86 86.3599 0)
 			(effects
@@
 			(project ""
 				(path "/4f9429d5-fbb3-48e9-90dd-7ff0c2950e6f/6b08732c-65b5-4020-967e-cc3e23d6bed3"
-					(reference "J35")
+					(reference "J34")
 					(unit 1)
 				)
@@
 		(dnp no)
 		(fields_autoplaced yes)
-		(property "Reference" "#PWR084"
+		(property "Reference" "#PWR082"
 			(at 128.27 80.01 0)
 			(effects
@@
 			(project ""
 				(path "/4f9429d5-fbb3-48e9-90dd-7ff0c2950e6f/6b08732c-65b5-4020-967e-cc3e23d6bed3"
-					(reference "#PWR084")
+					(reference "#PWR082")
 					(unit 1)
 				)
