File: hardware/PCB_Aquarium2/RasberryPi4.kicad_sch (KiCad schematic)
At the start: 2 parts, among them J34 Conn_01x04

Commit message: ajout des BOM
Parts:
- J34: footprint Connector_JST:JST_EH_B4B-EH-A_1x04_P2.50mm_Vertical -> Connector_JST:JST_XH_B4B-XH-A_1x04_P2.50mm_Vertical
Changed lines of the file:
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@@
 			)
 		)
-		(property "Footprint" "Connector_JST:JST_EH_B4B-EH-A_1x04_P2.50mm_Vertical"
+		(property "Footprint" "Connector_JST:JST_XH_B4B-XH-A_1x04_P2.50mm_Vertical"
 			(at 147.32 86.36 0)
 			(effects
