File: hardware/PCB_Aquarium2/Régulateur_de_tension.kicad_sch (KiCad schematic)
At the start: 10 parts, among them U2 173010578, U3 AZ1117-3.3

Commit message: PCBs v4
Parts:
- renumbered C11 to C38, C12 to C39, R3 to R5, R4 to R6, R5 to R7
Changed lines of the file:
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@@
 		(dnp no)
 		(fields_autoplaced yes)
-		(property "Reference" "#PWR072"
+		(property "Reference" "#PWR070"
 			(at 139.7 74.93 0)
 			(effects
@@
 			(project ""
 				(path "/4f9429d5-fbb3-48e9-90dd-7ff0c2950e6f/0b76def2-ce80-4218-8e3b-ba1c1b4e7345"
-					(reference "#PWR072")
+					(reference "#PWR070")
 					(unit 1)
 				)
@@
 		(dnp no)
 		(fields_autoplaced yes)
-		(property "Reference" "#PWR074"
+		(property "Reference" "#PWR072"
 			(at 139.7 107.95 0)
 			(effects
@@
 			(project ""
 				(path "/4f9429d5-fbb3-48e9-90dd-7ff0c2950e6f/0b76def2-ce80-4218-8e3b-ba1c1b4e7345"
-					(reference "#PWR074")
+					(reference "#PWR072")
 					(unit 1)
 				)
@@
 		(on_board yes)
 		(dnp no)
-		(property "Reference" "C12"
+		(property "Reference" "C39"
 			(at 154.94 83.8263 0)
 			(effects
@@
 			(project "PCB_Aquarium2"
 				(path "/4f9429d5-fbb3-48e9-90dd-7ff0c2950e6f/0b76def2-ce80-4218-8e3b-ba1c1b4e7345"
-					(reference "C12")
+					(reference "C39")
 					(unit 1)
 				)
@@
 		(on_board yes)
 		(dnp no)
-		(property "Reference" "R3"
+		(property "Reference" "R5"
 			(at 129.54 106.6799 0)
 			(effects
@@
 			(project "PCB_Aquarium2"
 				(path "/4f9429d5-fbb3-48e9-90dd-7ff0c2950e6f/0b76def2-ce80-4218-8e3b-ba1c1b4e7345"
-					(reference "R3")
+					(reference "R5")
 					(unit 1)
 				)
@@
 		(dnp no)
 		(fields_autoplaced yes)
-		(property "Reference" "R5"
+		(property "Reference" "R7"
 			(at 154.94 106.6799 0)
 			(effects
@@
 			(project "PCB_Aquarium2"
 				(path "/4f9429d5-fbb3-48e9-90dd-7ff0c2950e6f/0b76def2-ce80-4218-8e3b-ba1c1b4e7345"
-					(reference "R5")
+					(reference "R7")
 					(unit 1)
 				)
@@
 		(dnp no)
 		(fields_autoplaced yes)
-		(property "Reference" "#PWR075"
+		(property "Reference" "#PWR073"
 			(at 139.7 129.54 0)
 			(effects
@@
 			(project ""
 				(path "/4f9429d5-fbb3-48e9-90dd-7ff0c2950e6f/0b76def2-ce80-4218-8e3b-ba1c1b4e7345"
-					(reference "#PWR075")
+					(reference "#PWR073")
 					(unit 1)
 				)
@@
 		(dnp no)
 		(fields_autoplaced yes)
-		(property "Reference" "#PWR068"
+		(property "Reference" "#PWR066"
 			(at 121.92 86.36 0)
 			(effects
@@
 			(project ""
 				(path "/4f9429d5-fbb3-48e9-90dd-7ff0c2950e6f/0b76def2-ce80-4218-8e3b-ba1c1b4e7345"
-					(reference "#PWR068")
+					(reference "#PWR066")
 					(unit 1)
 				)
@@
 		(dnp no)
 		(fields_autoplaced yes)
-		(property "Reference" "#PWR076"
+		(property "Reference" "#PWR074"
 			(at 152.4 93.98 0)
 			(effects
@@
 			(project ""
 				(path "/4f9429d5-fbb3-48e9-90dd-7ff0c2950e6f/0b76def2-ce80-4218-8e3b-ba1c1b4e7345"
-					(reference "#PWR076")
+					(reference "#PWR074")
 					(unit 1)
 				)
@@
 		(dnp no)
 		(fields_autoplaced yes)
-		(property "Reference" "#PWR070"
+		(property "Reference" "#PWR068"
 			(at 125.73 93.98 0)
 			(effects
@@
 			(project ""
 				(path "/4f9429d5-fbb3-48e9-90dd-7ff0c2950e6f/0b76def2-ce80-4218-8e3b-ba1c1b4e7345"
-					(reference "#PWR070")
+					(reference "#PWR068")
 					(unit 1)
 				)
@@
 		(dnp no)
 		(fields_autoplaced yes)
-		(property "Reference" "#PWR073"
+		(property "Reference" "#PWR071"
 			(at 139.7 96.52 0)
 			(effects
@@
 			(project ""
 				(path "/4f9429d5-fbb3-48e9-90dd-7ff0c2950e6f/0b76def2-ce80-4218-8e3b-ba1c1b4e7345"
-					(reference "#PWR073")
+					(reference "#PWR071")
 					(unit 1)
 				)
@@
 		(dnp no)
 		(fields_autoplaced yes)
-		(property "Reference" "#PWR079"
+		(property "Reference" "#PWR077"
 			(at 156.21 86.36 0)
 			(effects
@@
 			(project "PCB_Aquarium2"
 				(path "/4f9429d5-fbb3-48e9-90dd-7ff0c2950e6f/0b76def2-ce80-4218-8e3b-ba1c1b4e7345"
-					(reference "#PWR079")
+					(reference "#PWR077")
 					(unit 1)
 				)
@@
 		(dnp no)
 		(fields_autoplaced yes)
-		(property "Reference" "#PWR078"
+		(property "Reference" "#PWR076"
 			(at 154.94 62.23 0)
 			(effects
@@
 			(project ""
 				(path "/4f9429d5-fbb3-48e9-90dd-7ff0c2950e6f/0b76def2-ce80-4218-8e3b-ba1c1b4e7345"
-					(reference "#PWR078")
+					(reference "#PWR076")
 					(unit 1)
 				)
@@
 		(dnp no)
 		(fields_autoplaced yes)
-		(property "Reference" "C11"
+		(property "Reference" "C38"
 			(at 128.27 83.8263 0)
 			(effects
@@
 			(project "PCB_Aquarium2"
 				(path "/4f9429d5-fbb3-48e9-90dd-7ff0c2950e6f/0b76def2-ce80-4218-8e3b-ba1c1b4e7345"
-					(reference "C11")
+					(reference "C38")
 					(unit 1)
 				)
@@
 		(dnp no)
 		(fields_autoplaced yes)
-		(property "Reference" "#PWR077"
+		(property "Reference" "#PWR075"
 			(at 152.4 107.95 0)
 			(effects
@@
 			(project "PCB_Aquarium2"
 				(path "/4f9429d5-fbb3-48e9-90dd-7ff0c2950e6f/0b76def2-ce80-4218-8e3b-ba1c1b4e7345"
-					(reference "#PWR077")
+					(reference "#PWR075")
 					(unit 1)
 				)
@@
 		(dnp no)
 		(fields_autoplaced yes)
-		(property "Reference" "R4"
+		(property "Reference" "R6"
 			(at 142.24 106.6799 0)
 			(effects
@@
 			(project "PCB_Aquarium2"
 				(path "/4f9429d5-fbb3-48e9-90dd-7ff0c2950e6f/0b76def2-ce80-4218-8e3b-ba1c1b4e7345"
-					(reference "R4")
+					(reference "R6")
 					(unit 1)
 				)
@@
 		(dnp no)
 		(fields_autoplaced yes)
-		(property "Reference" "#PWR071"
+		(property "Reference" "#PWR069"
 			(at 127 107.95 0)
 			(effects
@@
 			(project "PCB_Aquarium2"
 				(path "/4f9429d5-fbb3-48e9-90dd-7ff0c2950e6f/0b76def2-ce80-4218-8e3b-ba1c1b4e7345"
-					(reference "#PWR071")
+					(reference "#PWR069")
 					(unit 1)
 				)
@@
 		(dnp no)
 		(fields_autoplaced yes)
-		(property "Reference" "#PWR069"
+		(property "Reference" "#PWR067"
 			(at 123.19 60.96 0)
 			(effects
@@
 			(project "PCB_Aquarium2"
 				(path "/4f9429d5-fbb3-48e9-90dd-7ff0c2950e6f/0b76def2-ce80-4218-8e3b-ba1c1b4e7345"
-					(reference "#PWR069")
-					(unit 1)
-				)
+					(reference "#PWR067")
+					(unit 1)
+				)
