File: hardware/PCB_Aquarium2/STlink.kicad_sch (KiCad schematic)
At the start: 1 part, among them J36 Conn_ST_STDC14

Commit message: PCBs v4
Parts:
- renumbered J36 to J35
Changed lines of the file:
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@@
 		(dnp no)
 		(fields_autoplaced yes)
-		(property "Reference" "J36"
+		(property "Reference" "J35"
 			(at 128.27 93.9799 0)
 			(effects
@@
 			(project "PCB_Aquarium2"
 				(path "/4f9429d5-fbb3-48e9-90dd-7ff0c2950e6f/c9f60022-4980-4a06-8195-869d80fa4c60"
-					(reference "J36")
+					(reference "J35")
 					(unit 1)
 				)
@@
 		(dnp no)
 		(fields_autoplaced yes)
-		(property "Reference" "#PWR087"
+		(property "Reference" "#PWR085"
 			(at 139.7 121.92 0)
 			(effects
@@
 			(project "PCB_Aquarium2"
 				(path "/4f9429d5-fbb3-48e9-90dd-7ff0c2950e6f/c9f60022-4980-4a06-8195-869d80fa4c60"
-					(reference "#PWR087")
+					(reference "#PWR085")
 					(unit 1)
 				)
@@
 		(dnp no)
 		(fields_autoplaced yes)
-		(property "Reference" "#PWR086"
+		(property "Reference" "#PWR084"
 			(at 139.7 81.28 0)
 			(effects
@@
 			(project "PCB_Aquarium2"
 				(path "/4f9429d5-fbb3-48e9-90dd-7ff0c2950e6f/c9f60022-4980-4a06-8195-869d80fa4c60"
-					(reference "#PWR086")
+					(reference "#PWR084")
 					(unit 1)
 				)
