File: hardware/PCB_Aquarium2/Ventilateur.kicad_sch (KiCad schematic)
At the start: 1 part, among them J4 Conn_01x02

Commit message: PCBs v3
Parts:
- added C39: 1u, Capacitor_SMD:C_0603_1608Metric, symbol Device:C
Connections:
- net +12V: now also C39.1; no longer J4.1 (Pin_1)
- new net: C39.2, J4.1 (Pin_1)
Changed lines of the file:
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@@
-	(wire
-		(pts
-			(xy 143.51 106.68) (xy 144.78 106.68)
-		)
-		(stroke
-			(width 0)
-			(type default)
-		)
-	)
 	(wire
 		(pts
@@
 	)
 	(symbol
+		(lib_id "Device:C")
+		(at 140.97 106.68 90)
+		(unit 1)
+		(exclude_from_sim no)
+		(in_bom yes)
+		(on_board yes)
+		(dnp no)
+		(fields_autoplaced yes)
+		(property "Reference" "C39"
+			(at 140.97 99.06 90)
+			(effects
+				(font
+					(size 1.27 1.27)
+				)
+			)
+		)
+		(property "Value" "1u"
+			(at 140.97 101.6 90)
+			(effects
+				(font
+					(size 1.27 1.27)
+				)
+			)
+		)
+		(property "Footprint" "Capacitor_SMD:C_0603_1608Metric"
+			(at 144.78 105.7148 0)
+			(effects
+				(font
+					(size 1.27 1.27)
+				)
+				(hide yes)
+			)
+		)
+		(property "Datasheet" "~"
+			(at 140.97 106.68 0)
+			(effects
+				(font
+					(size 1.27 1.27)
+				)
+				(hide yes)
+			)
+		)
+		(property "Description" "Unpolarized capacitor"
+			(at 140.97 106.68 0)
+			(effects
+				(font
+					(size 1.27 1.27)
+				)
+				(hide yes)
+			)
+		)
+		(pin "1"
+		)
+		(pin "2"
+		)
+		(instances
+			(project ""
+				(path "/4f9429d5-fbb3-48e9-90dd-7ff0c2950e6f/b830814e-60b2-4976-ac6f-93ba76469b06/5d391acf-d6ea-4d4c-b787-b71a583dc165"
+					(reference "C39")
+					(unit 1)
+				)
+				(path "/4f9429d5-fbb3-48e9-90dd-7ff0c2950e6f/b830814e-60b2-4976-ac6f-93ba76469b06/d8f2eee3-0952-4164-a5fd-b230302140af"
+					(reference "C42")
+					(unit 1)
+				)
+				(path "/4f9429d5-fbb3-48e9-90dd-7ff0c2950e6f/b830814e-60b2-4976-ac6f-93ba76469b06/e3d823d5-1466-4ea5-81dd-ee852f5114d5"
+					(reference "C41")
+					(unit 1)
+				)
+				(path "/4f9429d5-fbb3-48e9-90dd-7ff0c2950e6f/b830814e-60b2-4976-ac6f-93ba76469b06/ea4cad06-5fb6-43d8-8ab4-a12c8caa015c"
+					(reference "C40")
+					(unit 1)
+				)
+			)
+		)
+	)
+	(symbol
 		(lib_id "power:+12V")
-		(at 143.51 106.68 0)
+		(at 137.16 106.68 0)
 		(unit 1)
 		(exclude_from_sim no)
@@
 		(fields_autoplaced yes)
 		(property "Reference" "#PWR012"
-			(at 143.51 110.49 0)
+			(at 137.16 110.49 0)
 			(effects
 				(font
@@
 		)
 		(property "Value" "+12V"
-			(at 143.51 101.6 0)
+			(at 137.16 101.6 0)
 			(effects
 				(font
@@
 		)
 		(property "Footprint" ""
-			(at 143.51 106.68 0)
+			(at 137.16 106.68 0)
 			(effects
 				(font
@@
 		)
 		(property "Datasheet" ""
-			(at 143.51 106.68 0)
+			(at 137.16 106.68 0)
 			(effects
 				(font
@@
 		)
 		(property "Description" "Power symbol creates a global label with name \"+12V\""
-			(at 143.51 106.68 0)
-			(effects
-				(font
+			(at 137.16 106.68 0)
+			(effects
+				(font

Commit message: PCBs v4
Parts:
- renumbered C39 to C12, J4 to J3
Connections:
- net +12V: now also C12.2, J3.1 (Pin_1); no longer C12.1
- net GND: now also C12.1
Other:
- moved on the sheet: C12
Changed lines of the file:
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@@
 	(generator_version "9.0")
 	(paper "A4")
-	(wire
-		(pts
-			(xy 143.51 109.22) (xy 144.78 109.22)
+	(junction
+		(at 140.97 114.3)
+		(diameter 0)
+		(color 0 0 0 0)
+	)
+	(junction
+		(at 140.97 106.68)
+		(diameter 0)
+		(color 0 0 0 0)
+	)
+	(wire
+		(pts
+			(xy 140.97 106.68) (xy 144.78 106.68)
+		)
+		(stroke
+			(width 0)
+			(type default)
+		)
+	)
+	(wire
+		(pts
+			(xy 144.78 114.3) (xy 144.78 109.22)
+		)
+		(stroke
+			(width 0)
+			(type default)
+		)
+	)
+	(wire
+		(pts
+			(xy 140.97 114.3) (xy 144.78 114.3)
+		)
+		(stroke
+			(width 0)
+			(type default)
+		)
+	)
+	(wire
+		(pts
+			(xy 137.16 114.3) (xy 140.97 114.3)
+		)
+		(stroke
+			(width 0)
+			(type default)
+		)
+	)
+	(wire
+		(pts
+			(xy 137.16 106.68) (xy 140.97 106.68)
 		)
 		(stroke
@@
 		(dnp no)
 		(fields_autoplaced yes)
-		(property "Reference" "J4"
+		(property "Reference" "J3"
 			(at 152.4 106.6799 0)
 			(effects
@@
 			(project "PCB_Aquarium2"
 				(path "/4f9429d5-fbb3-48e9-90dd-7ff0c2950e6f/b830814e-60b2-4976-ac6f-93ba76469b06/5d391acf-d6ea-4d4c-b787-b71a583dc165"
+					(reference "J3")
+					(unit 1)
+				)
+				(path "/4f9429d5-fbb3-48e9-90dd-7ff0c2950e6f/b830814e-60b2-4976-ac6f-93ba76469b06/d8f2eee3-0952-4164-a5fd-b230302140af"
+					(reference "J32")
+					(unit 1)
+				)
+				(path "/4f9429d5-fbb3-48e9-90dd-7ff0c2950e6f/b830814e-60b2-4976-ac6f-93ba76469b06/e3d823d5-1466-4ea5-81dd-ee852f5114d5"
+					(reference "J5")
+					(unit 1)
+				)
+				(path "/4f9429d5-fbb3-48e9-90dd-7ff0c2950e6f/b830814e-60b2-4976-ac6f-93ba76469b06/ea4cad06-5fb6-43d8-8ab4-a12c8caa015c"
 					(reference "J4")
-					(unit 1)
-				)
-				(path "/4f9429d5-fbb3-48e9-90dd-7ff0c2950e6f/b830814e-60b2-4976-ac6f-93ba76469b06/d8f2eee3-0952-4164-a5fd-b230302140af"
-					(reference "J33")
-					(unit 1)
-				)
-				(path "/4f9429d5-fbb3-48e9-90dd-7ff0c2950e6f/b830814e-60b2-4976-ac6f-93ba76469b06/e3d823d5-1466-4ea5-81dd-ee852f5114d5"
-					(reference "J6")
-					(unit 1)
-				)
-				(path "/4f9429d5-fbb3-48e9-90dd-7ff0c2950e6f/b830814e-60b2-4976-ac6f-93ba76469b06/ea4cad06-5fb6-43d8-8ab4-a12c8caa015c"
-					(reference "J5")
 					(unit 1)
 				)
@@
 	(symbol
 		(lib_id "power:GND")
-		(at 143.51 109.22 0)
+		(at 137.16 114.3 0)
 		(unit 1)
 		(exclude_from_sim no)
@@
 		(dnp no)
 		(fields_autoplaced yes)
-		(property "Reference" "#PWR013"
-			(at 143.51 115.57 0)
+		(property "Reference" "#PWR011"
+			(at 137.16 120.65 0)
 			(effects
 				(font
@@
 		)
 		(property "Value" "GND"
-			(at 143.51 114.3 0)
+			(at 137.16 119.38 0)
 			(effects
 				(font
@@
 		)
 		(property "Footprint" ""
-			(at 143.51 109.22 0)
+			(at 137.16 114.3 0)
 			(effects
 				(font
@@
 		)
 		(property "Datasheet" ""
-			(at 143.51 109.22 0)
+			(at 137.16 114.3 0)
 			(effects
 				(font
@@
 		)
 		(property "Description" "Power symbol creates a global label with name \"GND\" , ground"
-			(at 143.51 109.22 0)
+			(at 137.16 114.3 0)
 			(effects
 				(font
@@
 			(project "PCB_Aquarium2"
 				(path "/4f9429d5-fbb3-48e9-90dd-7ff0c2950e6f/b830814e-60b2-4976-ac6f-93ba76469b06/5d391acf-d6ea-4d4c-b787-b71a583dc165"
+					(reference "#PWR011")
+					(unit 1)
+				)
+				(path "/4f9429d5-fbb3-48e9-90dd-7ff0c2950e6f/b830814e-60b2-4976-ac6f-93ba76469b06/d8f2eee3-0952-4164-a5fd-b230302140af"
+					(reference "#PWR079")
+					(unit 1)
+				)
+				(path "/4f9429d5-fbb3-48e9-90dd-7ff0c2950e6f/b830814e-60b2-4976-ac6f-93ba76469b06/e3d823d5-1466-4ea5-81dd-ee852f5114d5"
+					(reference "#PWR015")
+					(unit 1)
+				)
+				(path "/4f9429d5-fbb3-48e9-90dd-7ff0c2950e6f/b830814e-60b2-4976-ac6f-93ba76469b06/ea4cad06-5fb6-43d8-8ab4-a12c8caa015c"
 					(reference "#PWR013")
-					(unit 1)
-				)
-				(path "/4f9429d5-fbb3-48e9-90dd-7ff0c2950e6f/b830814e-60b2-4976-ac6f-93ba76469b06/d8f2eee3-0952-4164-a5fd-b230302140af"
-					(reference "#PWR081")
-					(unit 1)
-				)
-				(path "/4f9429d5-fbb3-48e9-90dd-7ff0c2950e6f/b830814e-60b2-4976-ac6f-93ba76469b06/e3d823d5-1466-4ea5-81dd-ee852f5114d5"
-					(reference "#PWR017")
-					(unit 1)
-				)
-				(path "/4f9429d5-fbb3-48e9-90dd-7ff0c2950e6f/b830814e-60b2-4976-ac6f-93ba76469b06/ea4cad06-5fb6-43d8-8ab4-a12c8caa015c"
-					(reference "#PWR015")
 					(unit 1)
 				)
@@
 	(symbol
 		(lib_id "Device:C")
-		(at 140.97 106.68 90)
+		(at 140.97 110.49 180)
 		(unit 1)
 		(exclude_from_sim no)
@@
 		(dnp no)
 		(fields_autoplaced yes)
-		(property "Reference" "C39"
-			(at 140.97 99.06 90)
-			(effects
-				(font
-					(size 1.27 1.27)
-				)
+		(property "Reference" "C12"
+			(at 144.78 109.2199 0)
+			(effects
+				(font
+					(size 1.27 1.27)
+				)
+				(justify right)
 			)
 		)
 		(property "Value" "1u"
-			(at 140.97 101.6 90)
-			(effects
-				(font
-					(size 1.27 1.27)
-				)
+			(at 144.78 111.7599 0)
+			(effects
+				(font
+					(size 1.27 1.27)
+				)
+				(justify right)
 			)
 		)
 		(property "Footprint" "Capacitor_SMD:C_0603_1608Metric"
-			(at 144.78 105.7148 0)
+			(at 140.0048 106.68 0)
 			(effects
 				(font
@@
 		)
 		(property "Datasheet" "~"
-			(at 140.97 106.68 0)
+			(at 140.97 110.49 0)
 			(effects
 				(font
@@
 		)
 		(property "Description" "Unpolarized capacitor"
-			(at 140.97 106.68 0)
+			(at 140.97 110.49 0)
 			(effects
 				(font
@@
 		)
 		(instances
-			(project ""
+			(project "PCB_Aquarium2"
 				(path "/4f9429d5-fbb3-48e9-90dd-7ff0c2950e6f/b830814e-60b2-4976-ac6f-93ba76469b06/5d391acf-d6ea-4d4c-b787-b71a583dc165"
-					(reference "C39")
+					(reference "C12")
 					(unit 1)
 				)
 				(path "/4f9429d5-fbb3-48e9-90dd-7ff0c2950e6f/b830814e-60b2-4976-ac6f-93ba76469b06/d8f2eee3-0952-4164-a5fd-b230302140af"
-					(reference "C42")
+					(reference "C40")
 					(unit 1)
 				)
 				(path "/4f9429d5-fbb3-48e9-90dd-7ff0c2950e6f/b830814e-60b2-4976-ac6f-93ba76469b06/e3d823d5-1466-4ea5-81dd-ee852f5114d5"
-					(reference "C41")
+					(reference "C14")
 					(unit 1)
 				)
 				(path "/4f9429d5-fbb3-48e9-90dd-7ff0c2950e6f/b830814e-60b2-4976-ac6f-93ba76469b06/ea4cad06-5fb6-43d8-8ab4-a12c8caa015c"
-					(reference "C40")
+					(reference "C13")
 					(unit 1)
 				)
@@
 		(dnp no)
 		(fields_autoplaced yes)
-		(property "Reference" "#PWR012"
+		(property "Reference" "#PWR010"
 			(at 137.16 110.49 0)
 			(effects
@@
 			(project "PCB_Aquarium2"
 				(path "/4f9429d5-fbb3-48e9-90dd-7ff0c2950e6f/b830814e-60b2-4976-ac6f-93ba76469b06/5d391acf-d6ea-4d4c-b787-b71a583dc165"
+					(reference "#PWR010")
+					(unit 1)
+				)
+				(path "/4f9429d5-fbb3-48e9-90dd-7ff0c2950e6f/b830814e-60b2-4976-ac6f-93ba76469b06/d8f2eee3-0952-4164-a5fd-b230302140af"
+					(reference "#PWR078")
+					(unit 1)
+				)
+				(path "/4f9429d5-fbb3-48e9-90dd-7ff0c2950e6f/b830814e-60b2-4976-ac6f-93ba76469b06/e3d823d5-1466-4ea5-81dd-ee852f5114d5"
+					(reference "#PWR014")
+					(unit 1)
+				)
+				(path "/4f9429d5-fbb3-48e9-90dd-7ff0c2950e6f/b830814e-60b2-4976-ac6f-93ba76469b06/ea4cad06-5fb6-43d8-8ab4-a12c8caa015c"
 					(reference "#PWR012")
 					(unit 1)
 				)
-				(path "/4f9429d5-fbb3-48e9-90dd-7ff0c2950e6f/b830814e-60b2-4976-ac6f-93ba76469b06/d8f2eee3-0952-4164-a5fd-b230302140af"
-					(reference "#PWR080")
-					(unit 1)
-				)
-				(path "/4f9429d5-fbb3-48e9-90dd-7ff0c2950e6f/b830814e-60b2-4976-ac6f-93ba76469b06/e3d823d5-1466-4ea5-81dd-ee852f5114d5"
-					(reference "#PWR016")
-					(unit 1)
-				)
-				(path "/4f9429d5-fbb3-48e9-90dd-7ff0c2950e6f/b830814e-60b2-4976-ac6f-93ba76469b06/ea4cad06-5fb6-43d8-8ab4-a12c8caa015c"
-					(reference "#PWR014")
-					(unit 1)
-				)
