File: hardware/PCB_Aquarium2/Water_sensor.kicad_sch (KiCad schematic)
At the start: 3 parts, among them J25 Conn_01x03, J26 Conn_01x03, J27 Conn_01x03

Commit message: PCBs v3
Parts:
- added C25, C26, C27: 1u, Capacitor_SMD:C_0603_1608Metric, symbol Device:C
Connections:
- net +3.3V: now also C25.1, C26.1, C27.1; no longer J25.2 (Pin_2), J26.2 (Pin_2), J27.2 (Pin_2)
- new net: C25.2, J25.2 (Pin_2)
- new net: C26.2, J26.2 (Pin_2)
- new net: C27.2, J27.2 (Pin_2)

Commit message: PCBs v4
Parts:
- removed C25, C26: 1u, Capacitor_SMD:C_0603_1608Metric, symbol Device:C
- added C30, C31: 1u, Capacitor_SMD:C_0603_1608Metric, symbol Device:C
- renumbered C27 to C32, J25 to J24, J26 to J25, J27 to J26
Connections:
- net +3.3V: now also J24.2 (Pin_2), J25.2 (Pin_2), J26.2 (Pin_2), C30.1, C31.1
- net GND: now also C32.2, C30.2, C31.2
Other:
- moved on the sheet: C32
