File: hardware/PCB_Aquarium2/XT60.kicad_sch (KiCad schematic)
At the start: 2 parts, among them J34 Conn_01x02, SW2 SW_SPDT

Commit message: PCBs v4
Parts:
- renumbered J34 to J33
Changed lines of the file:
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@@
 		(dnp no)
 		(fields_autoplaced yes)
-		(property "Reference" "#PWR082"
+		(property "Reference" "#PWR080"
 			(at 137.16 99.06 0)
 			(effects
@@
 			(project ""
 				(path "/4f9429d5-fbb3-48e9-90dd-7ff0c2950e6f/abfb2004-d275-4aa1-bcad-0821a83fd301"
-					(reference "#PWR082")
+					(reference "#PWR080")
 					(unit 1)
 				)
@@
 		(dnp no)
 		(fields_autoplaced yes)
-		(property "Reference" "J34"
+		(property "Reference" "J33"
 			(at 130.81 78.74 0)
 			(effects
@@
 			(project "PCB_Aquarium2"
 				(path "/4f9429d5-fbb3-48e9-90dd-7ff0c2950e6f/abfb2004-d275-4aa1-bcad-0821a83fd301"
-					(reference "J34")
+					(reference "J33")
 					(unit 1)
 				)
@@
 		(dnp no)
 		(fields_autoplaced yes)
-		(property "Reference" "#PWR083"
+		(property "Reference" "#PWR081"
 			(at 153.67 85.09 0)
 			(effects
@@
 			(project "PCB_Aquarium2"
 				(path "/4f9429d5-fbb3-48e9-90dd-7ff0c2950e6f/abfb2004-d275-4aa1-bcad-0821a83fd301"
-					(reference "#PWR083")
+					(reference "#PWR081")
 					(unit 1)
 				)
