File: hardware/PCB_Aquarium2/screens_bouttons.kicad_sch (KiCad schematic)
At the start: 2 parts, among them J7 Conn_01x06, J8 Conn_01x06

Commit message: PCBs v3
Parts:
- added C36: 1u, Capacitor_SMD:C_0603_1608Metric, symbol Device:C
Connections:
- net +3.3V: now also C36.1; no longer J7.5 (Pin_5)
- new net: C36.2, J7.5 (Pin_5)
Changed lines of the file:
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@@
 	(wire
 		(pts
-			(xy 116.84 92.71) (xy 133.35 92.71)
+			(xy 125.73 92.71) (xy 133.35 92.71)
+		)
+		(stroke
+			(width 0)
+			(type default)
+		)
+	)
+	(wire
+		(pts
+			(xy 116.84 92.71) (xy 118.11 92.71)
 		)
 		(stroke
@@
 					(unit 1)
 				)
+			)
+		)
+	)
+	(symbol
+		(lib_id "Device:C")
+		(at 121.92 92.71 90)
+		(unit 1)
+		(exclude_from_sim no)
+		(in_bom yes)
+		(on_board yes)
+		(dnp no)
+		(fields_autoplaced yes)
+		(property "Reference" "C36"
+			(at 121.92 85.09 90)
+			(effects
+				(font
+					(size 1.27 1.27)
+				)
+			)
+		)
+		(property "Value" "1u"
+			(at 121.92 87.63 90)
+			(effects
+				(font
+					(size 1.27 1.27)
+				)
+			)
+		)
+		(property "Footprint" "Capacitor_SMD:C_0603_1608Metric"
+			(at 125.73 91.7448 0)
+			(effects
+				(font
+					(size 1.27 1.27)
+				)
+				(hide yes)
+			)
+		)
+		(property "Datasheet" "~"
+			(at 121.92 92.71 0)
+			(effects
+				(font
+					(size 1.27 1.27)
+				)
+				(hide yes)
+			)
+		)
+		(property "Description" "Unpolarized capacitor"
+			(at 121.92 92.71 0)
+			(effects
+				(font
+					(size 1.27 1.27)
+				)
+				(hide yes)
+			)
+		)
+		(pin "1"
+		)
+		(pin "2"
+		)
+		(instances
+			(project ""
+				(path "/4f9429d5-fbb3-48e9-90dd-7ff0c2950e6f/f32b2777-c21f-4b7d-8b68-c5d6df7ac0b7"
+					(reference "C36")
+					(unit 1)
+				)

Commit message: PCBs v4
Parts:
- renumbered C36 to C15, J7 to J6, J8 to J7
Connections:
- net +3.3V: now also C15.2, J6.5 (Pin_5); no longer C15.1
- net GND: now also C15.1
Other:
- moved on the sheet: C15
Changed lines of the file:
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@@
 	(generator_version "9.0")
 	(paper "A4")
+	(junction
+		(at 124.46 92.71)
+		(diameter 0)
+		(color 0 0 0 0)
+	)
+	(junction
+		(at 124.46 100.33)
+		(diameter 0)
+		(color 0 0 0 0)
+	)
 	(wire
 		(pts
-			(xy 130.81 95.25) (xy 133.35 95.25)
+			(xy 118.11 100.33) (xy 124.46 100.33)
 		)
 		(stroke
@@
 	(wire
 		(pts
-			(xy 125.73 92.71) (xy 133.35 92.71)
+			(xy 132.08 100.33) (xy 132.08 95.25)
 		)
 		(stroke
@@
 	(wire
 		(pts
-			(xy 116.84 92.71) (xy 118.11 92.71)
+			(xy 124.46 100.33) (xy 132.08 100.33)
 		)
 		(stroke
@@
 		)
 	)
+	(wire
+		(pts
+			(xy 132.08 95.25) (xy 133.35 95.25)
+		)
+		(stroke
+			(width 0)
+			(type default)
+		)
+	)
+	(wire
+		(pts
+			(xy 124.46 92.71) (xy 133.35 92.71)
+		)
+		(stroke
+			(width 0)
+			(type default)
+		)
+	)
+	(wire
+		(pts
+			(xy 116.84 92.71) (xy 124.46 92.71)
+		)
+		(stroke
+			(width 0)
+			(type default)
+		)
+	)
 	(hierarchical_label "SPI_SCK"
 		(shape input)
@@
 	(symbol
 		(lib_id "power:GND")
-		(at 130.81 95.25 0)
+		(at 118.11 100.33 0)
 		(unit 1)
 		(exclude_from_sim no)
@@
 		(dnp no)
 		(fields_autoplaced yes)
-		(property "Reference" "#PWR019"
-			(at 130.81 101.6 0)
+		(property "Reference" "#PWR017"
+			(at 118.11 106.68 0)
 			(effects
 				(font
@@
 		)
 		(property "Value" "GND"
-			(at 130.81 100.33 0)
+			(at 118.11 105.41 0)
 			(effects
 				(font
@@
 		)
 		(property "Footprint" ""
-			(at 130.81 95.25 0)
+			(at 118.11 100.33 0)
 			(effects
 				(font
@@
 		)
 		(property "Datasheet" ""
-			(at 130.81 95.25 0)
+			(at 118.11 100.33 0)
 			(effects
 				(font
@@
 		)
 		(property "Description" "Power symbol creates a global label with name \"GND\" , ground"
-			(at 130.81 95.25 0)
+			(at 118.11 100.33 0)
 			(effects
 				(font
@@
 			(project "PCB_Aquarium2"
 				(path "/4f9429d5-fbb3-48e9-90dd-7ff0c2950e6f/f32b2777-c21f-4b7d-8b68-c5d6df7ac0b7"
-					(reference "#PWR019")
+					(reference "#PWR017")
 					(unit 1)
 				)
@@
 	(symbol
 		(lib_id "Device:C")
-		(at 121.92 92.71 90)
+		(at 124.46 96.52 180)
 		(unit 1)
 		(exclude_from_sim no)
@@
 		(dnp no)
 		(fields_autoplaced yes)
-		(property "Reference" "C36"
-			(at 121.92 85.09 90)
-			(effects
-				(font
-					(size 1.27 1.27)
-				)
+		(property "Reference" "C15"
+			(at 128.27 95.2499 0)
+			(effects
+				(font
+					(size 1.27 1.27)
+				)
+				(justify right)
 			)
 		)
 		(property "Value" "1u"
-			(at 121.92 87.63 90)
-			(effects
-				(font
-					(size 1.27 1.27)
-				)
+			(at 128.27 97.7899 0)
+			(effects
+				(font
+					(size 1.27 1.27)
+				)
+				(justify right)
 			)
 		)
 		(property "Footprint" "Capacitor_SMD:C_0603_1608Metric"
-			(at 125.73 91.7448 0)
+			(at 123.4948 92.71 0)
 			(effects
 				(font
@@
 		)
 		(property "Datasheet" "~"
-			(at 121.92 92.71 0)
+			(at 124.46 96.52 0)
 			(effects
 				(font
@@
 		)
 		(property "Description" "Unpolarized capacitor"
-			(at 121.92 92.71 0)
+			(at 124.46 96.52 0)
 			(effects
 				(font
@@
 		)
 		(instances
-			(project ""
+			(project "PCB_Aquarium2"
 				(path "/4f9429d5-fbb3-48e9-90dd-7ff0c2950e6f/f32b2777-c21f-4b7d-8b68-c5d6df7ac0b7"
-					(reference "C36")
+					(reference "C15")
 					(unit 1)
 				)
@@
 		(dnp no)
 		(fields_autoplaced yes)
-		(property "Reference" "#PWR018"
+		(property "Reference" "#PWR016"
 			(at 116.84 96.52 0)
 			(effects
@@
 			(project "PCB_Aquarium2"
 				(path "/4f9429d5-fbb3-48e9-90dd-7ff0c2950e6f/f32b2777-c21f-4b7d-8b68-c5d6df7ac0b7"
-					(reference "#PWR018")
+					(reference "#PWR016")
 					(unit 1)
 				)
@@
 		(dnp no)
 		(fields_autoplaced yes)
-		(property "Reference" "J7"
+		(property "Reference" "J6"
 			(at 140.97 87.6299 0)
 			(effects
@@
 			(project ""
 				(path "/4f9429d5-fbb3-48e9-90dd-7ff0c2950e6f/f32b2777-c21f-4b7d-8b68-c5d6df7ac0b7"
-					(reference "J7")
+					(reference "J6")
 					(unit 1)
 				)
@@
 		(dnp no)
 		(fields_autoplaced yes)
-		(property "Reference" "J8"
+		(property "Reference" "J7"
 			(at 175.26 86.3599 0)
 			(effects
@@
 			(project "PCB_Aquarium2"
 				(path "/4f9429d5-fbb3-48e9-90dd-7ff0c2950e6f/f32b2777-c21f-4b7d-8b68-c5d6df7ac0b7"
-					(reference "J8")
+					(reference "J7")
 					(unit 1)
 				)
