File: hardware/PCB_Aquarium2/PCB_Aquarium2.kicad_pcb (KiCad board)
At the start: 4 copper layers, 71 x 61 mm, 69 parts, among them J1 Conn_01x03, J10 Conn_01x03, J11 Conn_01x03, J12 Conn_01x03, J13 Conn_01x03, J14 Conn_01x03, J15 Conn_01x03, J16 Conn_01x03, J17 Conn_01x03, J18 Conn_01x03, J19 Conn_01x03, J2 Conn_01x06, J20 Conn_01x03, J21 Conn_01x02, J22 Conn_01x02, J23 Conn_01x02, J24 Conn_01x02, J25 Conn_01x03, J26 Conn_01x03, J27 Conn_01x03, J28 Conn_01x03, J29 Conn_01x03, J30 Conn_01x03, J31 Conn_01x03, J32 Conn_01x03, J33 Conn_01x02, J34 Conn_01x02, J35 Conn_01x04, J36 Conn_ST_STDC14, J37 Conn_01x03, J38 Conn_01x03, J39 Conn_01x04, J4 Conn_01x02, J5 Conn_01x02, J6 Conn_01x02, J7 Conn_01x06, J8 Conn_01x06, J9 Conn_01x03, Q1 NPN, Q2 NPN, SW1 SW_SPST, SW2 SW_SPDT, U1 STM32G474RETx, U2 173010578, U3 AZ1117-3.3

Commit message: PCBs v2
Routing:
- net GND: vias 23 -> 48
Changed lines of the file:
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@@
+	)
+	(via
+		(at 124.39 117.4)
+		(size 0.45)
+		(drill 0.3)
+		(layers "F.Cu" "B.Cu")
+		(free yes)
+		(net 6)
+	)
+	(via
+		(at 149.59 108.43)
+		(size 0.45)
+		(drill 0.3)
+		(layers "F.Cu" "B.Cu")
+		(free yes)
+		(net 6)
 	)
 	(via
@@
 	)
 	(via
+		(at 116.93 125.51)
+		(size 0.45)
+		(drill 0.3)
+		(layers "F.Cu" "B.Cu")
+		(free yes)
+		(net 6)
+	)
+	(via
+		(at 182.75 98.35)
+		(size 0.45)
+		(drill 0.3)
+		(layers "F.Cu" "B.Cu")
+		(free yes)
+		(net 6)
+	)
+	(via
 		(at 144.25 93)
 		(size 0.45)
@@
 	)
 	(via
+		(at 154.5 76.7)
+		(size 0.45)
+		(drill 0.3)
+		(layers "F.Cu" "B.Cu")
+		(free yes)
+		(net 6)
+	)
+	(via
+		(at 149.59 115.77)
+		(size 0.45)
+		(drill 0.3)
+		(layers "F.Cu" "B.Cu")
+		(free yes)
+		(net 6)
+	)
+	(via
+		(at 117.14 99.33)
+		(size 0.45)
+		(drill 0.3)
+		(layers "F.Cu" "B.Cu")
+		(free yes)
+		(net 6)
+	)
+	(via
+		(at 156.48 107.96)
+		(size 0.45)
+		(drill 0.3)
+		(layers "F.Cu" "B.Cu")
+		(free yes)
+		(net 6)
+	)
+	(via
 		(at 124.315669 119.331796)
 		(size 0.45)
@@
 	)
 	(via
+		(at 119 105.19)
+		(size 0.45)
+		(drill 0.3)
+		(layers "F.Cu" "B.Cu")
+		(free yes)
+		(net 6)
+	)
+	(via
 		(at 157.75 95.425)
 		(size 0.45)
@@
 	)
 	(via
+		(at 170.94 115.93)
+		(size 0.45)
+		(drill 0.3)
+		(layers "F.Cu" "B.Cu")
+		(free yes)
+		(net 6)
+	)
+	(via
+		(at 134.58 80.99)
+		(size 0.45)
+		(drill 0.3)
+		(layers "F.Cu" "B.Cu")
+		(free yes)
+		(net 6)
+	)
+	(via
 		(at 153.55 116.05)
 		(size 0.45)
@@
 	)
 	(via
+		(at 123.97 113.02)
+		(size 0.45)
+		(drill 0.3)
+		(layers "F.Cu" "B.Cu")
+		(free yes)
+		(net 6)
+	)
+	(via
+		(at 179.23 84.7)
+		(size 0.45)
+		(drill 0.3)
+		(layers "F.Cu" "B.Cu")
+		(free yes)
+		(net 6)
+	)
+	(via
 		(at 163.5 116.9)
 		(size 0.45)
@@
 	)
 	(via
+		(at 116.64 117.56)
+		(size 0.45)
+		(drill 0.3)
+		(layers "F.Cu" "B.Cu")
+		(free yes)
+		(net 6)
+	)
+	(via
 		(at 165.05 76.3)
 		(size 0.45)
@@
 	)
 	(via
+		(at 125.3 75.54)
+		(size 0.45)
+		(drill 0.3)
+		(layers "F.Cu" "B.Cu")
+		(free yes)
+		(net 6)
+	)
+	(via
 		(at 158.44 93.076)
 		(size 0.45)
@@
 	)
 	(via
+		(at 184.48 123.37)
+		(size 0.45)
+		(drill 0.3)
+		(layers "F.Cu" "B.Cu")
+		(free yes)
+		(net 6)
+	)
+	(via
+		(at 140.69 93.8)
+		(size 0.45)
+		(drill 0.3)
+		(layers "F.Cu" "B.Cu")
+		(free yes)
+		(net 6)
+	)
+	(via
 		(at 162.51 76.3)
 		(size 0.45)
@@
 	)
 	(via
+		(at 124.1 132.31)
+		(size 0.45)
+		(drill 0.3)
+		(layers "F.Cu" "B.Cu")
+		(free yes)
+		(net 6)
+	)
+	(via
+		(at 117.23 90.78)
+		(size 0.45)
+		(drill 0.3)
+		(layers "F.Cu" "B.Cu")
+		(free yes)
+		(net 6)
+	)
+	(via
 		(at 141.8 101.9)
 		(size 0.45)
@@
 	)
 	(via
+		(at 182.32 113.37)
+		(size 0.45)
+		(drill 0.3)
+		(layers "F.Cu" "B.Cu")
+		(free yes)
+		(net 6)
+	)
+	(via
 		(at 123.2 124.3875)
 		(size 0.45)
@@
 	)
 	(via
+		(at 176.46 75.82)
+		(size 0.45)
+		(drill 0.3)
+		(layers "F.Cu" "B.Cu")
+		(free yes)
+		(net 6)
+	)
+	(via
+		(at 180.11 105.58)
+		(size 0.45)
+		(drill 0.3)
+		(layers "F.Cu" "B.Cu")
+		(free yes)
+		(net 6)
+	)
+	(via
+		(at 127.11 79.69)
+		(size 0.45)
+		(drill 0.3)
+		(layers "F.Cu" "B.Cu")
+		(free yes)
+		(net 6)
+	)
+	(via
 		(at 176.55 97.55)
 		(size 0.45)
@@
 		(net 6)
 	)
+	(via
+		(at 117.26 109.34)
+		(size 0.45)
+		(drill 0.3)
+		(layers "F.Cu" "B.Cu")
+		(free yes)
+		(net 6)
+	)
+	(via
+		(at 173.25 78.99)
+		(size 0.45)
+		(drill 0.3)
+		(layers "F.Cu" "B.Cu")
+		(free yes)
+		(net 6)
+	)

Commit message: PCBs v3
Parts:
- removed J21: Conn_01x02, Connector_JST:JST_EH_B2B-EH-A_1x02_P2.50mm_Vertical
- removed Q1, Q2: NPN, Package_TO_SOT_SMD:TSOT-23
- removed R1, R2: 240, Resistor_SMD:R_0805_2012Metric
- added C13: 1u, Capacitor_SMD:C_0603_1608Metric, B.Cu at (128.3, 87.2)
- added C14: 1u, Capacitor_SMD:C_0603_1608Metric, B.Cu at (123.8, 87.2)
- added C15: 1u, Capacitor_SMD:C_0603_1608Metric, B.Cu at (118.8, 87.0)
- added C16: 1u, Capacitor_SMD:C_0603_1608Metric, B.Cu at (118.6, 98.9)
- added C17: 1u, Capacitor_SMD:C_0603_1608Metric, B.Cu at (182.0, 118.6)
- added C18: 1u, Capacitor_SMD:C_0603_1608Metric, B.Cu at (175.1, 109.7)
- added C19: 1u, Capacitor_SMD:C_0603_1608Metric, B.Cu at (128.1, 98.2)
- added C20: 1u, Capacitor_SMD:C_0603_1608Metric, B.Cu at (178.7, 102.6)
- added C21: 1u, Capacitor_SMD:C_0603_1608Metric, B.Cu at (141.3, 105.0)
- added C22: 1u, Capacitor_SMD:C_0603_1608Metric, B.Cu at (131.2, 115.8)
- added C23: 1u, Capacitor_SMD:C_0603_1608Metric, B.Cu at (141.1, 114.0)
- added C24: 1u, Capacitor_SMD:C_0603_1608Metric, B.Cu at (152.3, 113.8)
- added C25: 1u, Capacitor_SMD:C_0603_1608Metric, B.Cu at (154.7, 84.1)
- added C26: 1u, Capacitor_SMD:C_0603_1608Metric, B.Cu at (159.7, 82.7)
- added C27: 1u, Capacitor_SMD:C_0603_1608Metric, B.Cu at (147.4, 81.2)
- added C28: 1u, Capacitor_SMD:C_0603_1608Metric, B.Cu at (134.2, 87.4)
- added C29: 1u, Capacitor_SMD:C_0603_1608Metric, B.Cu at (160.6, 89.6)
- added C30: 1u, Capacitor_SMD:C_0603_1608Metric, B.Cu at (147.2, 90.5)
- added C31: 1u, Capacitor_SMD:C_0603_1608Metric, B.Cu at (130.1, 106.1)
- added C32: 1u, Capacitor_SMD:C_0603_1608Metric, B.Cu at (133.4, 98.8)
- added C33: 1u, Capacitor_SMD:C_0603_1608Metric, B.Cu at (165.7, 89.2)
- added C34: 1u, Capacitor_SMD:C_0603_1608Metric, B.Cu at (123.2, 98.2)
- added C35: 1u, Capacitor_SMD:C_0603_1608Metric, B.Cu at (173.6, 101.8)
- added C36: 1u, Capacitor_SMD:C_0603_1608Metric, B.Cu at (145.0, 79.0)
- added C37: 1u, Capacitor_SMD:C_0603_1608Metric, B.Cu at (170.9, 87.6)
- added C38: 1u, Capacitor_SMD:C_0603_1608Metric, B.Cu at (118.8, 109.7)
- added C39: 1u, Capacitor_SMD:C_0603_1608Metric, B.Cu at (165.2, 132.1)
- added C40: 1u, Capacitor_SMD:C_0603_1608Metric, B.Cu at (173.3, 122.9)
- added C41: 1u, Capacitor_SMD:C_0603_1608Metric, B.Cu at (175.9, 128.8)
- added C42: 1u, Capacitor_SMD:C_0603_1608Metric, B.Cu at (158.2, 131.9)
- added C43: 1u, Capacitor_SMD:C_0603_1608Metric, B.Cu at (157.3, 127.2)
- added C44: 1u, Capacitor_SMD:C_0603_1608Metric, B.Cu at (167.0, 127.2)
- added J40: Conn_01x02, Connector_JST:JST_EH_B2B-EH-A_1x02_P2.50mm_Vertical, F.Cu at (157.4, 120.0)
- added L1: 39n, Inductor_SMD:L_0805_2012Metric, F.Cu at (140.5, 102.4)
- added Q3: NMOS, Package_TO_SOT_SMD:SOT-23, F.Cu at (166.2, 116.1)
- added Q4: NMOS, Package_TO_SOT_SMD:SOT-23, F.Cu at (160.1, 116.1)
- added R6: 1k, Resistor_SMD:R_0402_1005Metric, F.Cu at (169.3, 115.1)
- added R7: 10k, Resistor_SMD:R_0402_1005Metric, F.Cu at (169.3, 117.1)
- added R8: 1k, Resistor_SMD:R_0402_1005Metric, F.Cu at (163.1, 115.1)
- added R9: 10k, Resistor_SMD:R_0402_1005Metric, F.Cu at (163.2, 117.2)
- C1, C10, C5: footprint Capacitor_SMD:C_0402_1005Metric -> Capacitor_SMD:C_0603_1608Metric
- moved J6 12.4 mm to (174.0, 129.6), turned to 90 degrees
- moved J22 12.3 mm to (166.2, 120.0), turned to 0 degrees
- moved C10 11.6 mm to (153.2, 107.2), turned to 180 degrees
- moved C9 9.76 mm to (143.5, 102.4), turned to 90 degrees
- moved C1 1.73 mm to (158.4, 93.6)
- moved C5 1.43 mm to (142.2, 102.5)
- moved C3 1.07 mm to (156.6, 93.6)
- moved C6 1.05 mm to (152.7, 105.9)
Connections:
- J1 pad 2: +5V -> Net-(J1-Pin_2)
- J1 pad 3: GPIO_PH -> ADC1_IN10_PH
- J10 pad 2: +5V -> Net-(J10-Pin_2)
- J11 pad 2: +5V -> Net-(J11-Pin_2)
- J12 pad 2: +5V -> Net-(J12-Pin_2)
- J13 pad 2: +5V -> Net-(J13-Pin_2)
- J14 pad 2: +5V -> Net-(J14-Pin_2)
- J15 pad 2: +5V -> Net-(J15-Pin_2)
- J16 pad 2: +5V -> Net-(J16-Pin_2)
- J17 pad 2: +5V -> Net-(J17-Pin_2)
- J18 pad 2: +5V -> Net-(J18-Pin_2)
- J19 pad 2: +5V -> Net-(J19-Pin_2)
- J20 pad 2: +5V -> Net-(J20-Pin_2)
- J22 pad 2: GND -> Net-(J22-Pin_2)
- J23 pad 1: +12V -> Net-(J23-Pin_1)
- J24 pad 1: +12V -> Net-(J24-Pin_1)
- J25 pad 2: +3.3V -> Net-(J25-Pin_2)
- J26 pad 2: +3.3V -> Net-(J26-Pin_2)
- J27 pad 2: +3.3V -> Net-(J27-Pin_2)
- J28 pad 1: +5V -> Net-(J28-Pin_1)
- J29 pad 2: +5V -> Net-(J29-Pin_2)
- J30 pad 2: +5V -> Net-(J30-Pin_2)
- J31 pad 2: +5V -> Net-(J31-Pin_2)
- J32 pad 2: +5V -> Net-(J32-Pin_2)
- J33 pad 1: +12V -> Net-(J33-Pin_1)
- J35 pad 1: +5V -> Net-(J35-Pin_1)
- J37 pad 1: +5V -> Net-(J37-Pin_1)
- J38 pad 2: +5V -> Net-(J38-Pin_2)
- J39 pad 1: +5V -> Net-(J39-Pin_1)
- J4 pad 1: +12V -> Net-(J4-Pin_1)
- J5 pad 1: +12V -> Net-(J5-Pin_1)
- J6 pad 1: +12V -> Net-(J6-Pin_1)
- J7 pad 5: +3.3V -> Net-(J7-Pin_5)
- J9 pad 2: +5V -> Net-(J9-Pin_2)
- U1 pad 2: GPIO_PH -> unconnected-(U1-PC13-Pad2)
- U1 pad 5: unconnected-(U1-PF0-Pad5) -> ADC1_IN10_PH
Routing:
- net +5V: track 9.20 -> 32.3 mm, vias 2 -> 24
- net ADC1_IN10_PH: track 0.00 -> 14.7 mm, vias 0 -> 2
- net +3.3V: track 28.3 -> 40.5 mm, vias 9 -> 13
- net GPIO_PH: track 11.2 -> 0.00 mm
- net GPIO_PUMP_2: track 18.3 -> 23.7 mm
- net Net-(Q3-G): track 0.00 -> 5.12 mm
- net Net-(Q2-B): track 4.54 -> 0.00 mm
- net Net-(J27-Pin_2): track 0.00 -> 3.75 mm, vias 0 -> 1
- net Net-(Q4-G): track 0.00 -> 3.71 mm
- net Net-(J22-Pin_2): track 0.00 -> 3.64 mm
- net GPIO_PUMP_1: track 16.4 -> 20.0 mm
- net Net-(J40-Pin_2): track 0.00 -> 3.47 mm
- net Net-(J14-Pin_2): track 0.00 -> 3.12 mm
- net Net-(J31-Pin_2): track 0.00 -> 3.06 mm
- net Net-(J10-Pin_2): track 0.00 -> 2.98 mm
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Other:
- board text added: "+12V +5V +3.3V"

Commit message: PCBs v4
Parts:
- removed the C13 at (128.3, 87.2)
- removed the C14 at (123.8, 87.2)
- removed the C15 at (118.8, 87.0)
- removed the C25 at (154.7, 84.1)
- removed the C26 at (159.7, 82.7)
- removed the C44 at (167.0, 127.2)
- removed J39: Conn_01x04, Connector_JST:JST_EH_B4B-EH-A_1x04_P2.50mm_Vertical
- removed J40: Conn_01x02, Connector_JST:JST_EH_B2B-EH-A_1x02_P2.50mm_Vertical
- removed Q3, Q4: NMOS, Package_TO_SOT_SMD:SOT-23
- removed R8: 1k, Resistor_SMD:R_0402_1005Metric
- removed R9: 10k, Resistor_SMD:R_0402_1005Metric
- added C21: 1u, Capacitor_SMD:C_0603_1608Metric, B.Cu at (129.1, 97.2)
- added C22: 1u, Capacitor_SMD:C_0603_1608Metric, B.Cu at (181.6, 118.3)
- added C23: 1u, Capacitor_SMD:C_0603_1608Metric, B.Cu at (175.6, 109.7)
- added C29: 1u, Capacitor_SMD:C_0603_1608Metric, B.Cu at (158.7, 127.1)
- added C30: 1u, Capacitor_SMD:C_0603_1608Metric, B.Cu at (150.7, 84.0)
- added C31: 1u, Capacitor_SMD:C_0603_1608Metric, B.Cu at (155.6, 84.1)
- added J20: Conn_01x02, Connector_JST:JST_EH_B2B-EH-A_1x02_P2.50mm_Vertical, F.Cu at (157.5, 120.0)
- added J38: Conn_01x04, Connector_JST:JST_EH_B4B-EH-A_1x04_P2.50mm_Vertical, F.Cu at (121.2, 108.7)
- added Q1: NMOS, Package_TO_SOT_SMD:SOT-23, F.Cu at (160.0, 116.1)
- added Q2: NMOS, Package_TO_SOT_SMD:SOT-23, F.Cu at (166.0, 116.1)
- added R1: 1k, Resistor_SMD:R_0402_1005Metric, F.Cu at (162.9, 115.1)
- added R2: 10k, Resistor_SMD:R_0402_1005Metric, F.Cu at (162.9, 117.3)
- moved C17 66.6 mm to (118.9, 97.5), turned to 90 degrees
- moved C18 51.5 mm to (129.0, 86.8), turned to 90 degrees
- moved C19 15.1 mm to (118.8, 86.3), turned to 90 degrees
- moved C16 13.7 mm to (124.1, 86.3), turned to 90 degrees
- moved C28 10.1 mm to (167.4, 127.3), turned to 180 degrees
- moved C13 4.06 mm to (175.8, 119.7), turned to -90 degrees
- moved C32 2.42 mm to (145.0, 81.0), turned to 0 degrees
- moved C12 2.24 mm to (167.5, 132.0), turned to 180 degrees
- moved C37 2.07 mm to (128.1, 106.0)
- moved C24 2.02 mm to (139.3, 105.0)
- moved C36 1.91 mm to (134.2, 97.0)
- moved C11 1.58 mm to (134.1, 85.9)
- moved C42 1.27 mm to (173.7, 103.1)
- moved C34 1.00 mm to (123.9, 97.5), turned to 90 degrees
- moved C14 0.63 mm to (176.0, 128.2)
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- renumbered C28 to C11, C39 to C12, C40 to C13, C41 to C14, C36 to C15, C21 to C24, C23 to C25, C22 to C26, C24 to C27, C43 to C28, C27 to C32, C30 to C33, C33 to C35, C32 to C36, C31 to C37, C11 to C38, C12 to C39, C42 to C40, C37 to C41, C35 to C42, C29 to C43, C38 to C44, J11 to J10, J12 to J11, J13 to J12, J14 to J13, J16 to J14, J17 to J16, J19 to J17, J20 to J19, J22 to J21, J23 to J22, J24 to J23, J25 to J24, J26 to J25, J27 to J26, J28 to J27, J29 to J28, J30 to J29, J4 to J3, J31 to J30, J32 to J31, J33 to J32, J34 to J33, J35 to J34, J36 to J35, J37 to J36, J38 to J37, J5 to J4, J6 to J5, J7 to J6, J8 to J7, J9 to J8, J10 to J9, R6 to R3, R7 to R4, R3 to R5, R4 to R6, R5 to R7
Connections:
- C11 pad 2: Net-(J1-Pin_2) -> GND
- C12 pad 1: +12V -> GND
- C12 pad 2: Net-(J4-Pin_1) -> +12V
- C13 pad 1: +12V -> GND
- C13 pad 2: Net-(J5-Pin_1) -> +12V
- C14 pad 1: +12V -> GND
- C14 pad 2: Net-(J6-Pin_1) -> +12V
- C15 pad 1: +3.3V -> GND
- C15 pad 2: Net-(J7-Pin_5) -> +3.3V
- C16 pad 2: Net-(J9-Pin_2) -> GND
- C17 pad 2: Net-(J16-Pin_2) -> GND
- C18 pad 2: Net-(J15-Pin_2) -> GND
- C19 pad 2: Net-(J14-Pin_2) -> GND
- C20 pad 2: Net-(J13-Pin_2) -> GND
- C24 pad 2: Net-(J17-Pin_2) -> GND
- C25 pad 1: +5V -> GND
- C25 pad 2: Net-(J19-Pin_2) -> +5V
- C26 pad 1: +5V -> GND
- C26 pad 2: Net-(J18-Pin_2) -> +5V
- C27 pad 2: Net-(J20-Pin_2) -> GND
- C28 pad 1: +12V -> GND
- C28 pad 2: Net-(J23-Pin_1) -> +12V
- C32 pad 2: Net-(J27-Pin_2) -> GND
- C33 pad 1: +5V -> GND
- C33 pad 2: Net-(J28-Pin_1) -> +5V
- C34 pad 2: Net-(J29-Pin_2) -> GND
- C35 pad 2: Net-(J30-Pin_2) -> GND
- C36 pad 2: Net-(J31-Pin_2) -> GND
- C37 pad 2: Net-(J32-Pin_2) -> GND
- C40 pad 1: +12V -> GND
- C40 pad 2: Net-(J33-Pin_1) -> +12V
- C41 pad 1: +5V -> GND
- C41 pad 2: Net-(J35-Pin_1) -> +5V
- C42 pad 1: +5V -> GND
- C42 pad 2: Net-(J37-Pin_1) -> +5V
- C43 pad 2: Net-(J38-Pin_2) -> GND
- C44 pad 1: +5V -> GND
- C44 pad 2: Net-(J39-Pin_1) -> +5V
- J1 pad 2: Net-(J1-Pin_2) -> +5V
- J10 pad 2: Net-(J11-Pin_2) -> +5V
- J11 pad 2: Net-(J12-Pin_2) -> +5V
- J12 pad 2: Net-(J13-Pin_2) -> +5V
- J13 pad 2: Net-(J14-Pin_2) -> +5V
- J14 pad 2: Net-(J16-Pin_2) -> +5V
- J15 pad 2: Net-(J15-Pin_2) -> +5V
- J16 pad 2: Net-(J17-Pin_2) -> +5V
- J17 pad 2: Net-(J19-Pin_2) -> +5V
- J18 pad 2: Net-(J18-Pin_2) -> +5V
- J19 pad 2: Net-(J20-Pin_2) -> +5V
- J22 pad 1: Net-(J23-Pin_1) -> +12V
- J23 pad 1: Net-(J24-Pin_1) -> +12V
- J24 pad 2: Net-(J25-Pin_2) -> +3.3V
- J25 pad 2: Net-(J26-Pin_2) -> +3.3V
- J26 pad 2: Net-(J27-Pin_2) -> +3.3V
- J27 pad 1: Net-(J28-Pin_1) -> +5V
- J28 pad 2: Net-(J29-Pin_2) -> +5V
- J29 pad 2: Net-(J30-Pin_2) -> +5V
- J3 pad 1: Net-(J4-Pin_1) -> +12V
- J30 pad 2: Net-(J31-Pin_2) -> +5V
- J31 pad 2: Net-(J32-Pin_2) -> +5V
- J32 pad 1: Net-(J33-Pin_1) -> +12V
- J34 pad 1: Net-(J35-Pin_1) -> +5V
- J36 pad 1: Net-(J37-Pin_1) -> +5V
- J37 pad 2: Net-(J38-Pin_2) -> +5V
- J4 pad 1: Net-(J5-Pin_1) -> +12V
- J5 pad 1: Net-(J6-Pin_1) -> +12V
- J6 pad 5: Net-(J7-Pin_5) -> +3.3V
- J8 pad 2: Net-(J9-Pin_2) -> +5V
- J9 pad 2: Net-(J10-Pin_2) -> +5V
Routing:
- net GND: track 39.9 -> 109.3 mm, vias 49 -> 51
- net +5V: track 32.3 -> 59.4 mm, vias 24 -> 2
- net +12V: track 6.92 -> 14.3 mm, vias 7 -> 1
- net +3.3V: track 40.5 -> 45.1 mm, vias 13 -> 9
- net Net-(J27-Pin_2): track 3.75 -> 0.00 mm, vias 1 -> 0
- net Net-(Q1-G): track 0.00 -> 3.75 mm
- net Net-(Q4-G): track 3.71 -> 0.00 mm
- net Net-(J40-Pin_2): track 3.47 -> 0.00 mm
- net Net-(J14-Pin_2): track 3.12 -> 0.00 mm
- net Net-(J31-Pin_2): track 3.06 -> 0.00 mm
- net Net-(J10-Pin_2): track 2.98 -> 0.00 mm
- net Net-(J29-Pin_2): track 2.84 -> 0.00 mm
- net Net-(J26-Pin_2): track 2.61 -> 0.00 mm
- net Net-(J9-Pin_2): track 2.61 -> 0.00 mm
- net Net-(J7-Pin_5): track 2.48 -> 0.00 mm
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Other:
- board text added: "GPIOs BTNs"
- board text added: "HC05"
- board text added: "LED 5VDC"
- board text added: "MOTEURS 12V"
- board text added: "PI4"
- board text added: "SERVOMOTEURS 5VDC"
- board text added: "SPI(1) 3.3VDC"
- board text added: "SPI(2) CS 1-6"
- board text added: "WATER SENSORS 5V"

Commit message: PCBs V5
Routing:
- net +3.3V: track 45.1 -> 45.4 mm, vias 9 -> 11
Changed lines of the file:
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@@
+	(segment
+		(start 140.46 103.43)
+		(end 139.35 103.43)
+		(width 0.2)
+		(layer "F.Cu")
+		(net 1)
+	)
 	(segment
 		(start 140.46 103.43)
@@
 	)
 	(segment
-		(start 140.46 101.305)
-		(end 140.46 102.36)
-		(width 0.2)
-		(layer "F.Cu")
-		(net 1)
-	)
-	(segment
 		(start 143.54 102.85)
 		(end 144.12 102.85)
@@
 	)
 	(segment
+		(start 139.85 101.305)
+		(end 139.33 101.825)
+		(width 0.2)
+		(layer "F.Cu")
+		(net 1)
+	)
+	(segment
 		(start 145.06 93.93)
 		(end 146.11 92.88)
@@
 	)
 	(segment
+		(start 140.46 101.305)
+		(end 139.85 101.305)
+		(width 0.2)
+		(layer "F.Cu")
+		(net 1)
+	)
+	(segment
 		(start 153.15 105.93)
 		(end 153.15 106.385)
@@
 	)
 	(segment
-		(start 140.46 102.36)
-		(end 140.46 103.43)
-		(width 0.2)
-		(layer "F.Cu")
-		(net 1)
-	)
-	(segment
 		(start 142.03 103.43)
 		(end 142.18 103.28)
@@
 	)
 	(via
+		(at 139.33 101.825)
+		(size 0.45)
+		(drill 0.3)
+		(layers "F.Cu" "B.Cu")
+		(net 1)
+	)
+	(via
 		(at 158.395958 95.352608)
 		(size 0.45)
@@
 		(size 0.45)
 		(drill 0.3)
+		(layers "F.Cu" "B.Cu")
+		(net 1)
+	)
+	(via
+		(at 139.35 103.43)
+		(size 0.45)
+		(drill 0.3)
