File: hardware/PCB_secondaire/PCB_secondaire.kicad_pcb (KiCad board)
At the start: 2 copper layers, 72 x 28 mm, 35 parts, among them J1 Conn_01x07, J2 Conn_01x06, J3 Conn_01x07, J4 Conn_01x07, J5 Conn_01x07, J6 Conn_01x07, J7 Conn_01x06, J8 Conn_01x06, J9 Conn_01x07, SW1 SW_SPST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

Commit message: PCBs v2
Parts:
- J3, J4, J5: footprint Connector_PinHeader_2.54mm:PinHeader_1x07_P2.54mm_Vertical -> Connector_PinHeader_2.54mm:PinHeader_1x07_P2.54mm_Horizontal
- moved J3 70.0 mm to (99.0, 129.1)
- moved J5 68.1 mm to (147.0, 129.1)
- moved R3 63.3 mm to (110.6, 147.0)
- moved C2 63.3 mm to (112.5, 147.0)
- moved SW2 63.3 mm to (112.6, 143.1)
- moved R4 63.3 mm to (114.5, 147.0)
- moved R7 61.8 mm to (134.7, 147.0)
- moved C4 61.8 mm to (136.7, 147.0)
- moved R8 61.7 mm to (138.7, 147.0)
- moved SW4 61.7 mm to (136.6, 143.1)
- moved SW1 57.1 mm to (100.6, 143.1)
- moved R1 57.1 mm to (98.6, 147.0)
- moved C1 57.0 mm to (100.6, 147.0)
- moved R2 57.0 mm to (102.6, 147.0)
- moved R12 56.5 mm to (164.1, 147.0)
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Routing:
- net /SPI_D/C: track 0.00 -> 86.9 mm
- net /SPI_MOSI: track 0.00 -> 86.0 mm
- net /SPI_RES: track 0.00 -> 84.6 mm, vias 0 -> 2
- net /SPI_SCK: track 0.00 -> 83.8 mm, vias 0 -> 2
- net BTN_1: track 0.00 -> 48.1 mm
- net BTN_2: track 0.00 -> 40.2 mm, vias 0 -> 2
- net /SPI_CS_2: track 0.00 -> 37.8 mm
- net /SPI_CS_1: track 0.00 -> 35.4 mm, vias 0 -> 1
- net /SPI_CS_5: track 0.00 -> 32.9 mm
- net BTN_3: track 0.00 -> 31.7 mm, vias 0 -> 2
- net /SPI_CS_4: track 0.00 -> 25.2 mm
- net /SPI_CS_6: track 0.00 -> 22.6 mm
- net /SPI_CS_3: track 0.00 -> 21.8 mm
- net GND: track 0.00 -> 19.8 mm, vias 0 -> 104
- net BTN_4: track 0.00 -> 16.9 mm, vias 0 -> 2
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- added copper zone on In2.Cu, net +3.3V
- added copper zone on B.Cu, net GND
- added copper zone on F.Cu, net GND
- added copper zone on In1.Cu, net GND
Other:
- board size 72 x 28 mm -> 72 x 31.1 mm
- copper layers 2 -> 4

Commit message: PCBs v3
Parts:
- added C10: 1u, Capacitor_SMD:C_0603_1608Metric, F.Cu at (116.9, 129.4)
- added C11: 1u, Capacitor_SMD:C_0603_1608Metric, F.Cu at (136.5, 135.7)
- added C12: 1u, Capacitor_SMD:C_0603_1608Metric, F.Cu at (160.4, 135.7)
- added C7: 1u, Capacitor_SMD:C_0603_1608Metric, F.Cu at (112.5, 135.6)
- added C8: 1u, Capacitor_SMD:C_0603_1608Metric, F.Cu at (140.9, 131.1)
- added C9: 1u, Capacitor_SMD:C_0603_1608Metric, F.Cu at (164.9, 129.5)
Connections:
- J1 pad 6: +3.3V -> Net-(J1-Pin_6)
- J3 pad 6: +3.3V -> Net-(J3-Pin_6)
- J4 pad 6: +3.3V -> Net-(J4-Pin_6)
- J5 pad 6: +3.3V -> Net-(J5-Pin_6)
- J6 pad 6: +3.3V -> Net-(J6-Pin_6)
- J9 pad 6: +3.3V -> Net-(J9-Pin_6)
Routing:
- net +3.3V: track 4.83 -> 11.3 mm, vias 6 -> 12
- net Net-(J3-Pin_6): track 0.00 -> 5.86 mm
- net Net-(J4-Pin_6): track 0.00 -> 5.72 mm
- net Net-(J5-Pin_6): track 0.00 -> 5.66 mm
- net Net-(J6-Pin_6): track 0.00 -> 2.69 mm
- net Net-(J9-Pin_6): track 0.00 -> 2.66 mm
- net Net-(J1-Pin_6): track 0.00 -> 2.65 mm
- net /SPI_CS_1: track 35.4 -> 36.1 mm

Commit message: PCBs v4
Parts:
- moved C8 1.78 mm to (140.9, 129.3)
- turned C10 to -90 degrees
- turned C11 to 180 degrees
- turned C12 to 180 degrees
- turned C7 to 180 degrees
- turned C9 to -90 degrees
Connections:
- C10 pad 1: Net-(J3-Pin_6) -> GND
- C11 pad 1: Net-(J6-Pin_6) -> GND
- C12 pad 1: Net-(J9-Pin_6) -> GND
- C7 pad 1: Net-(J1-Pin_6) -> GND
- C8 pad 1: Net-(J4-Pin_6) -> GND
- C9 pad 1: Net-(J5-Pin_6) -> GND
- J1 pad 6: Net-(J1-Pin_6) -> +3.3V
- J3 pad 6: Net-(J3-Pin_6) -> +3.3V
- J4 pad 6: Net-(J4-Pin_6) -> +3.3V
- J5 pad 6: Net-(J5-Pin_6) -> +3.3V
- J6 pad 6: Net-(J6-Pin_6) -> +3.3V
- J9 pad 6: Net-(J9-Pin_6) -> +3.3V
Routing:
- net +3.3V: track 11.3 -> 30.0 mm, vias 12 -> 6
- net GND: track 19.8 -> 25.7 mm, vias 104 -> 109
- net Net-(J3-Pin_6): track 5.86 -> 0.00 mm
- net Net-(J4-Pin_6): track 5.72 -> 0.00 mm
- net Net-(J5-Pin_6): track 5.66 -> 0.00 mm
- net Net-(J6-Pin_6): track 2.69 -> 0.00 mm
- net Net-(J9-Pin_6): track 2.66 -> 0.00 mm
- net Net-(J1-Pin_6): track 2.65 -> 0.00 mm
